File: designs/rpi-mains-relay/out/ch2.kicad_sch (KiCad schematic)
At the start: 8 parts, among them J3 2606-3102/020-000, K2 G5RL-1A-E-TV8 DC5, Q2 AO3400A

Commit message: designs: work-in-progress (Prius encoding and relay-board rework under way)
Co-Authored-By: Claude Opus 5.5 <noreply@anthropic.com>
Claude-Session: https://claude.ai/code/session_01VFJn9VbX8h27kf4LpLwEtn
Parts:
- removed D6: green, LED_SMD:LED_0603_1608Metric, symbol Device:LED
- removed J3: 2606-3102/020-000, custom:WAGO_2606-3102_020-000, symbol Connector_Generic:Conn_01x02
- removed R10: 1.5k, Resistor_SMD:R_0603_1608Metric, symbol Device:R
- removed R6: 4.7k, Resistor_SMD:R_0603_1608Metric, symbol Device:R
- added D8: green, LED_SMD:LED_0603_1608Metric, symbol Device:LED
- added R14: 1.5k, Resistor_SMD:R_0603_1608Metric, symbol Device:R
- added R8: 4.7k, Resistor_SMD:R_0603_1608Metric, symbol Device:R
- R2: value 1k -> 100; MPN RC0603FR-071KL -> RC0603FR-07100RL
Connections:
- net +5V: now also R14.1
- net CH2_G: now also R8.1
- net COIL2: now also D8.1 (K)
- net GND: now also R8.2
- net LED2_A: now also D8.2 (A), R14.2
- net CH2_IN renamed CH2
Other:
- title: Channel 2: relay K2, driver Q2, output J3 -> Outlet 2: relay K2, driver Q2
- moved on the sheet: R2
Changed lines of the file:
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@@
 	(paper "A4")
 	(title_block
-		(title "Channel 2: relay K2, driver Q2, output J3")
+		(title "Outlet 2: relay K2, driver Q2")
 		(date "2026-10-23")
 		(rev "A")
 		(company "kaesynth")
-		(comment 1 "CH2_IN = Pi pin 13 (BCM27); K2 switches L_IN to L_SW2; J3 = OUT2 L/N")
-		(comment 2 "RPi 4-channel 120 VAC relay board (4-11/16 in box) — generated by kaesynth from design.py; do not edit by hand")
+		(comment 1 "CH2 = Pi pin 13 (BCM27); K2 switches L_IN to L_SW2 -> J2.3")
+		(comment 2 "RPi Zero 2 W six-outlet 120 VAC relay board (polycarbonate enclosure) — generated by kaesynth from design.py; do not edit by hand")
 	)
 	(symbol
 		(lib_id "Device:R")
-		(at 27.94 96.52 0)
+		(at 27.94 93.98 0)
 		(unit 1)
 		(exclude_from_sim no)
@@
 		(dnp no)
 		(property "Reference" "R2"
-			(at 29.972 96.52 90)
-			(effects
-				(font (size 1.27 1.27))
-			)
-		)
-		(property "Value" "1k"
-			(at 27.94 96.52 90)
+			(at 29.972 93.98 90)
+			(effects
+				(font (size 1.27 1.27))
+			)
+		)
+		(property "Value" "100"
+			(at 27.94 93.98 90)
 			(effects
 				(font (size 1.27 1.27))
@@
 		)
 		(property "Footprint" "Resistor_SMD:R_0603_1608Metric"
-			(at 27.94 96.52 0)
+			(at 27.94 93.98 0)
 			(hide yes)
 			(effects
@@
 		)
 		(property "Datasheet" "https://yageogroup.com/content/datasheet/asset/file/PYU-RC_GROUP_51_ROHS_L"
-			(at 27.94 96.52 0)
-			(hide yes)
-			(effects
-				(font (size 1.27 1.27))
-			)
-		)
-		(property "Description" "Resistor 1k 1% 0603"
-			(at 27.94 96.52 0)
-			(hide yes)
-			(effects
-				(font (size 1.27 1.27))
-			)
-		)
-		(property "MPN" "RC0603FR-071KL"
-			(at 27.94 96.52 0)
+			(at 27.94 93.98 0)
+			(hide yes)
+			(effects
+				(font (size 1.27 1.27))
+			)
+		)
+		(property "Description" "Resistor 100 1% 0603"
+			(at 27.94 93.98 0)
+			(hide yes)
+			(effects
+				(font (size 1.27 1.27))
+			)
+		)
+		(property "MPN" "RC0603FR-07100RL"
+			(at 27.94 93.98 0)
 			(hide yes)
 			(effects
@@
 		)
 		(property "Manufacturer" "YAGEO"
-			(at 27.94 96.52 0)
+			(at 27.94 93.98 0)
 			(hide yes)
 			(effects
@@
 		)
 		(property "Block" "ch2"
-			(at 27.94 96.52 0)
+			(at 27.94 93.98 0)
 			(hide yes)
 			(effects
@@
 		)
 		(property "Component Class" "ch2"
-			(at 27.94 96.52 0)
+			(at 27.94 93.98 0)
 			(hide yes)
 			(effects
@@
 		)
 		(property "Tolerance" "1%"
-			(at 27.94 96.52 0)
+			(at 27.94 93.98 0)
 			(hide yes)
 			(effects
@@
 		)
 		(property "Package" "0603"
-			(at 27.94 96.52 0)
+			(at 27.94 93.98 0)
 			(hide yes)
 			(effects
@@
 	)
 	(wire
-		(pts (xy 27.94 92.71) (xy 27.94 90.17))
-		(stroke
-			(width 0)
-			(type default)
-		)
-	)
-	(global_label "CH2_IN"
+		(pts (xy 27.94 90.17) (xy 27.94 87.63))
+		(stroke
+			(width 0)
+			(type default)
+		)
+	)
+	(global_label "CH2"
 		(shape passive)
-		(at 27.94 90.17 90)
+		(at 27.94 87.63 90)
 		(fields_autoplaced yes)
 		(effects
@@
 		)
 		(property "Intersheetrefs" "${INTERSHEET_REFS}"
-			(at 27.94 90.17 0)
-			(hide yes)
-			(effects
-				(font (size 1.27 1.27))
-			)
-		)
-	)
-	(wire
-		(pts (xy 27.94 100.33) (xy 27.94 102.87))
+			(at 27.94 87.63 0)
+			(hide yes)
+			(effects
+				(font (size 1.27 1.27))
+			)
+		)
+	)
+	(wire
+		(pts (xy 27.94 97.79) (xy 27.94 100.33))
 		(stroke
 			(width 0)
@@
 	)
 	(label "CH2_G"
-		(at 27.94 102.87 270)
+		(at 27.94 100.33 270)
 		(fields_autoplaced yes)
 		(effects
@@
 		(on_board yes)
 		(dnp no)
-		(property "Reference" "R6"
+		(property "Reference" "R8"
 			(at 42.672 96.52 90)
 			(effects
@@
 			(project "rpi-mains-relay"
 				(path "/a30cabb5-b934-5e97-9aeb-aaefec3ba07a/6de384ee-328d-5456-b0b0-d4b97d794c0d"
-					(reference "R6")
+					(reference "R8")
 					(unit 1)
 				)
@@
 		(on_board yes)
 		(dnp no)
-		(property "Reference" "D6"
+		(property "Reference" "D8"
 			(at 66.04 78.74 0)
 			(effects
@@
 			(project "rpi-mains-relay"
 				(path "/a30cabb5-b934-5e97-9aeb-aaefec3ba07a/6de384ee-328d-5456-b0b0-d4b97d794c0d"
-					(reference "D6")
+					(reference "D8")
 					(unit 1)
 				)
@@
 		(on_board yes)
 		(dnp no)
-		(property "Reference" "R10"
+		(property "Reference" "R14"
 			(at 136.652 96.52 90)
 			(effects
@@
 			(project "rpi-mains-relay"
 				(path "/a30cabb5-b934-5e97-9aeb-aaefec3ba07a/6de384ee-328d-5456-b0b0-d4b97d794c0d"
-					(reference "R10")
+					(reference "R14")
 					(unit 1)
 				)
@@
 		)
 	)
-	(symbol
-		(lib_id "Connector_Generic:Conn_01x02")
-		(at 162.56 83.82 0)
-		(unit 1)
-		(exclude_from_sim no)
-		(in_bom yes)
-		(on_board yes)
-		(dnp no)
-		(property "Reference" "J3"
-			(at 162.56 81.28 0)
-			(effects
-				(font (size 1.27 1.27))
-			)
-		)
-		(property "Value" "2606-3102/020-000"
-			(at 162.56 88.9 0)
-			(effects
-				(font (size 1.27 1.27))
-			)
-		)
-		(property "Footprint" "custom:WAGO_2606-3102_020-000"
-			(at 162.56 83.82 0)
-			(hide yes)
-			(effects
-				(font (size 1.27 1.27))
-			)
-		)
-		(property "Datasheet" "https://www.wago.com/2606-3102/020-000"
-			(at 162.56 83.82 0)
-			(hide yes)
-			(effects
-				(font (size 1.27 1.27))
-			)
-		)
-		(property "Description" "PCB terminal block 2-pole, lever, push-in CAGE CLAMP, 6 mm2, 7.5 mm pitch, staggered pins"
-			(at 162.56 83.82 0)
-			(hide yes)
-			(effects
-				(font (size 1.27 1.27))
-			)
-		)
-		(property "MPN" "2606-3102/020-000"
-			(at 162.56 83.82 0)
-			(hide yes)
-			(effects
-				(font (size 1.27 1.27))
-			)
-		)
-		(property "Manufacturer" "WAGO"
-			(at 162.56 83.82 0)
-			(hide yes)
-			(effects
-				(font (size 1.27 1.27))
-			)
-		)
-		(property "Block" "ch2"
-			(at 162.56 83.82 0)
-			(hide yes)
-			(effects
-				(font (size 1.27 1.27))
-			)
-		)
-		(property "Component Class" "ch2"
-			(at 162.56 83.82 0)
-			(hide yes)
-			(effects
-				(font (size 1.27 1.27))
-			)
-		)
-		(pin "1"
-		)
-		(pin "2"
-		)
-		(instances
-			(project "rpi-mains-relay"
-				(path "/a30cabb5-b934-5e97-9aeb-aaefec3ba07a/6de384ee-328d-5456-b0b0-d4b97d794c0d"
-					(reference "J3")
-					(unit 1)
-				)
-			)
-		)
-	)
-	(wire
-		(pts (xy 157.48 83.82) (xy 154.94 83.82))
-		(stroke
-			(width 0)
-			(type default)
-		)
-	)
-	(global_label "L_SW2"
-		(shape passive)
-		(at 154.94 83.82 180)
-		(fields_autoplaced yes)
-		(effects
-			(font (size 1.27 1.27))
-			(justify right)
-		)
-		(property "Intersheetrefs" "${INTERSHEET_REFS}"
-			(at 154.94 83.82 0)
-			(hide yes)
-			(effects
-				(font (size 1.27 1.27))
-			)
-		)
-	)
-	(wire
-		(pts (xy 157.48 86.36) (xy 154.94 86.36))
-		(stroke
-			(width 0)
-			(type default)
-		)
-	)
-	(global_label "N"
-		(shape passive)
-		(at 154.94 86.36 180)
-		(fields_autoplaced yes)
-		(effects
-			(font (size 1.27 1.27))
-			(justify right)
-		)
-		(property "Intersheetrefs" "${INTERSHEET_REFS}"
-			(at 154.94 86.36 0)
-			(hide yes)
-			(effects
-				(font (size 1.27 1.27))
-			)
-		)
-	)
