File: designs/rpi-mains-relay/out/mains_in.kicad_sch (KiCad schematic)
At the start: 1 part, among them J1 2606-3102/020-000

Commit message: designs: work-in-progress (Prius encoding and relay-board rework under way)
Co-Authored-By: Claude Opus 5.5 <noreply@anthropic.com>
Claude-Session: https://claude.ai/code/session_01VFJn9VbX8h27kf4LpLwEtn
Parts:
- added F1: 1A, Fuse:Fuseholder_Clip-6.3x32mm_Littelfuse_102071_Inline_P34.70x7.60mm_D2.00mm_Horizontal, symbol Device:Fuse
- added PS1: IRM-20-5, Converter_ACDC:Converter_ACDC_MeanWell_IRM-20-xx_THT, symbol Converter_ACDC:IRM-20-5
Connections:
- net L_IN: now also F1.1
- net N: now also PS1.2 (AC/N)
- new net +5V: PS1.4 (+Vo)
- new net GND: PS1.3 (-Vo)
- new net L_PSU: F1.2, PS1.1 (AC/L)
Other:
- title: Mains input terminal (shared L, N) -> Mains input J1, supply fuse F1 and IRM-20-5
- moved on the sheet: J1
