File: designs/rpi-mains-relay/out/pi.kicad_sch (KiCad schematic)
At the start: 4 parts, among them J5 PPPC202LFBN-RC

Commit message: designs/rpi-mains-relay: work-in-progress rework (6 receptacles, Pi Zero 2 W inside)
Co-Authored-By: Claude Opus 5.5 <noreply@anthropic.com>
Claude-Session: https://claude.ai/code/session_01VFJn9VbX8h27kf4LpLwEtn
Changed lines of the file:
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@@
 		(company "kaesynth")
 		(comment 1 "J5 back-feeds 5 V on pins 2/4; 3V3 from pins 1/17 powers U1; antenna zone keepout")
-		(comment 2 "RPi Zero 2 W six-outlet 120 VAC relay board (polycarbonate enclosure) — generated by kaesynth from design.py; do not edit by hand")
+		(comment 2 "RPi Zero 2 W 6-outlet 120 VAC relay board — generated by kaesynth from design.py; do not edit by hand")
 	)
 	(symbol
@@
 		)
 	)
-	(label "ARM_FB"
+	(global_label "ARM_FB"
+		(shape passive)
 		(at 53.34 73.66 0)
 		(fields_autoplaced yes)
@@
 			(justify left)
 		)
-	)
+		(property "Intersheetrefs" "${INTERSHEET_REFS}"
+			(at 53.34 73.66 0)
+			(hide yes)
+			(effects
+				(font (size 1.27 1.27))
+			)
+		)
+	)
