File: designs/rpi-mains-relay/out/outlets.kicad_sch (KiCad schematic)
At the start: 3 parts, among them J2 2606-3103/020-000, J3 2606-3103/020-000, J4 2606-3103/020-000

Commit message: designs/rpi-mains-relay: revision 3 — one enclosure (user decision)
User chose one enclosure (2026-10-23, Q-8). An ABB/Carlon NS14126 polycarbonate UL 50
Type 4X enclosure (14 x 12 x 6 in; Wi-Fi passes) holds the unchanged 200 x 150 mm board on
its back panel; three split-tab TR duplex receptacles mount in a 3-gang cut-out in the
cover on a 6.4 mm polycarbonate subplate, yokes bonded by pigtails, 14 AWG leads with a
service loop to J2-J4. A partition keeps receptacles and field wiring away from the board's
SELV side; the Pi is >= 150 mm from them. 15.5 W gives 49 C inside at a 40 C room.

No listed nonmetallic enclosure with receptacle openings in its cover was found, so
cover-mounted receptacles need a field evaluation or a UL 508A shop: new blocking Q-17.
All mains barriers ac=True. Build: 0 errors, 0 warnings, 31 waived, ERC clean, netlist
identical (L_IN now correctly flagged: relays sit on the wire side of the supply fuse;
the branch-breaker waiver covers it).

Co-Authored-By: Claude Opus 5.5 <noreply@anthropic.com>
Claude-Session: https://claude.ai/code/session_01VFJn9VbX8h27kf4LpLwEtn
Other:
- title: Receptacle feeds J2-J4 (one 14/3 NM-B cable per duplex receptacle) -> Receptacle feeds J2-J4 (three 14 AWG leads per duplex receptacle in the cover)
Changed lines of the file:
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@@
 	(paper "A4")
 	(title_block
-		(title "Receptacle feeds J2-J4 (one 14/3 NM-B cable per duplex receptacle)")
+		(title "Receptacle feeds J2-J4 (three 14 AWG leads per duplex receptacle in the cover)")
 		(date "2026-10-23")
 		(rev "A")
