File: designs/rpi-mains-relay/out/arm.kicad_sch (KiCad schematic)
At the start: 10 parts, among them Q5 AO3400A

Commit message: designs: work-in-progress (Prius encoding and relay-board rework under way)
Co-Authored-By: Claude Opus 5.5 <noreply@anthropic.com>
Claude-Session: https://claude.ai/code/session_01VFJn9VbX8h27kf4LpLwEtn
Parts:
- removed C3: 1u, Capacitor_SMD:C_0603_1608Metric, symbol Device:C
- removed C4: 100n, Capacitor_SMD:C_0603_1608Metric, symbol Device:C
- removed D12: BAT54S, Package_TO_SOT_SMD:SOT-23, symbol Diode:BAT54S
- removed D9: green, LED_SMD:LED_0603_1608Metric, symbol Device:LED
- removed Q5: AO3400A, Package_TO_SOT_SMD:SOT-23, symbol Transistor_FET:AO3400A
- removed R13: 1k, Resistor_SMD:R_0603_1608Metric, symbol Device:R
- removed R14: 1M, Resistor_SMD:R_0603_1608Metric, symbol Device:R
- removed R15: 1.5k, Resistor_SMD:R_0603_1608Metric, symbol Device:R
- added C6, C7: 100n, Capacitor_SMD:C_0603_1608Metric, symbol Device:C
- added D13: green, LED_SMD:LED_0603_1608Metric, symbol Device:LED
- added D16: BAT54S, Package_TO_SOT_SMD:SOT-23, symbol Diode:BAT54S
- added Q7: AO3400A, Package_TO_SOT_SMD:SOT-23, symbol Transistor_FET:AO3400A
- added R19: 1.5k, Resistor_SMD:R_0603_1608Metric, symbol Device:R
- added R21: 330k, Resistor_SMD:R_0603_1608Metric, symbol Device:R
- added R22, R23: 100k, Resistor_SMD:R_0603_1608Metric, symbol Device:R
- added R24: 47k, Resistor_SMD:R_0603_1608Metric, symbol Device:R
- added R25: 68k, Resistor_SMD:R_0603_1608Metric, symbol Device:R
- added R26: 10k, Resistor_SMD:R_0603_1608Metric, symbol Device:R
- added TP5: TP, TestPoint:TestPoint_Pad_D1.5mm, symbol Connector:TestPoint
- added U1: 74LVC1G123, Package_SO:SSOP-8_2.95x2.8mm_P0.65mm, symbol 74xGxx:74LVC1G123
Connections:
- net +5V: now also R19.1, R26.1
- net ARM_G: now also Q7.1 (G), R22.1, U1.5 (Q)
- net COIL_RTN: now also D13.1 (K), Q7.3 (D), R24.1, R26.2
- net GND: now also C7.2, D16.1 (A), Q7.2 (S), R22.2, R23.2, R25.2, U1.1 (~{A}), U1.4 (GND)
- net LED_ARM_A: now also D13.2 (A), R19.2
- new net +3V3: C7.1, D16.2 (K), R21.1, U1.3 (~{CLR}), U1.8 (VCC)
- new net ARM_FB: D16.3 (COM), R24.2, R25.1
- new net HB: R23.1, TP5.1, U1.2 (B)
- new net WD_CX: C6.2, U1.6 (Cext)
- new net WD_RC: C6.1, R21.2, U1.7 (RCext)
Other:
- title: Heartbeat watchdog (charge pump) and common coil enable -> Heartbeat watchdog U1, arming switch Q7 and readback
- moved on the sheet: TP3, TP4

Commit message: designs/rpi-mains-relay: work-in-progress rework (6 receptacles, Pi Zero 2 W inside)
Co-Authored-By: Claude Opus 5.5 <noreply@anthropic.com>
Claude-Session: https://claude.ai/code/session_01VFJn9VbX8h27kf4LpLwEtn
Changed lines of the file:
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@@
 		(company "kaesynth")
 		(comment 1 "Q7 closes the coil return only while HB has rising edges; OFF <= 0.1 s after they stop")
-		(comment 2 "RPi Zero 2 W six-outlet 120 VAC relay board (polycarbonate enclosure) — generated by kaesynth from design.py; do not edit by hand")
+		(comment 2 "RPi Zero 2 W 6-outlet 120 VAC relay board — generated by kaesynth from design.py; do not edit by hand")
 	)
 	(symbol
@@
 		)
 	)
-	(label "ARM_FB"
+	(global_label "ARM_FB"
+		(shape passive)
 		(at 226.06 87.63 270)
 		(fields_autoplaced yes)
@@
 			(font (size 1.27 1.27))
 			(justify right)
+		)
+		(property "Intersheetrefs" "${INTERSHEET_REFS}"
+			(at 226.06 87.63 0)
+			(hide yes)
+			(effects
+				(font (size 1.27 1.27))
+			)
 		)
 	)
@@
 		)
 	)
-	(label "ARM_FB"
+	(global_label "ARM_FB"
+		(shape passive)
 		(at 236.22 72.39 90)
 		(fields_autoplaced yes)
@@
 			(font (size 1.27 1.27))
 			(justify left)
+		)
+		(property "Intersheetrefs" "${INTERSHEET_REFS}"
+			(at 236.22 72.39 0)
+			(hide yes)
+			(effects
+				(font (size 1.27 1.27))
+			)
 		)
 	)
@@
 		)
 	)
-	(label "ARM_FB"
+	(global_label "ARM_FB"
+		(shape passive)
 		(at 241.3 38.1 270)
 		(fields_autoplaced yes)
@@
 			(justify right)
 		)
-	)
+		(property "Intersheetrefs" "${INTERSHEET_REFS}"
+			(at 241.3 38.1 0)
+			(hide yes)
+			(effects
+				(font (size 1.27 1.27))
+			)
+		)
+	)

Commit message: designs/rpi-mains-relay: fix the revision-3 re-review findings
- Watchdog: turn-off back to <= 0.5 s (no source asked for faster); R21 1 M, C6 220 nF
  give a 150-340 ms window. wdsim.py (a time-domain model used by design.py's calcs):
  stuck high/low off in 165-356 ms, heartbeat gaps up to 152 ms ride through, chatter
  only at 2.9-6.7 Hz; heartbeat >= 20 Hz from a priority thread; test plan corrected.
- Finger-safe polycarbonate shield over the supply fuse, relay contacts, supply AC pins
  and line copper; receptacle backs shrouded.
- Cover receptacles: brass threaded inserts, fine-stranded 14 AWG leads with ferrules and
  strain relief, 20 N pull test; the field cut drops the enclosure to Type 1 (indoor dry),
  stated in Q-17.
- Minors fixed or answered. Build: 0 errors, ERC clean, netlist identical, 31 waived.

Co-Authored-By: Claude Opus 5.5 <noreply@anthropic.com>
Claude-Session: https://claude.ai/code/session_01VFJn9VbX8h27kf4LpLwEtn
Parts:
- C6: value 100n -> 220n; MPN CC0603KRX7R9BB104 -> CC0603KRX7R9BB224
- R21: value 330k -> 1M; MPN RC0603FR-07330KL -> RC0603FR-071ML
Changed lines of the file:
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@@
 		(rev "A")
 		(company "kaesynth")
-		(comment 1 "Q7 closes the coil return only while HB has rising edges; OFF <= 0.1 s after they stop")
+		(comment 1 "Q7 closes the coil return only while HB has rising edges; OFF <= 0.36 s after they stop")
 		(comment 2 "RPi Zero 2 W 6-outlet 120 VAC relay board — generated by kaesynth from design.py; do not edit by hand")
 	)
@@
 			)
 		)
-		(property "Value" "330k"
+		(property "Value" "1M"
 			(at 27.94 88.9 90)
 			(effects
@@
 			)
 		)
-		(property "Description" "Resistor 330k 1% 0603"
-			(at 27.94 88.9 0)
-			(hide yes)
-			(effects
-				(font (size 1.27 1.27))
-			)
-		)
-		(property "MPN" "RC0603FR-07330KL"
+		(property "Description" "Resistor 1M 1% 0603"
+			(at 27.94 88.9 0)
+			(hide yes)
+			(effects
+				(font (size 1.27 1.27))
+			)
+		)
+		(property "MPN" "RC0603FR-071ML"
 			(at 27.94 88.9 0)
 			(hide yes)
@@
 			)
 		)
-		(property "Value" "100n"
+		(property "Value" "220n"
 			(at 41.275 91.44 0)
 			(effects
@@
 			)
 		)
-		(property "Description" "Capacitor 100n 50V X7R 0603"
+		(property "Description" "Capacitor 220n 50V X7R 0603"
 			(at 40.64 88.9 0)
 			(hide yes)
@@
 			)
 		)
-		(property "MPN" "CC0603KRX7R9BB104"
+		(property "MPN" "CC0603KRX7R9BB224"
 			(at 40.64 88.9 0)
 			(hide yes)
