File: designs/rpi-mains-relay/out/mech.kicad_sch (KiCad schematic)
At the start: 12 parts

Commit message: designs: work-in-progress (Prius encoding and relay-board rework under way)
Co-Authored-By: Claude Opus 5.5 <noreply@anthropic.com>
Claude-Session: https://claude.ai/code/session_01VFJn9VbX8h27kf4LpLwEtn
Parts:
- added H10, H7, H8, H9: MountingHole, MountingHole:MountingHole_2.7mm_M2.5, symbol Mechanical:MountingHole
- added H5, H6: MountingHole, MountingHole:MountingHole_3.2mm_M3, symbol Mechanical:MountingHole
- added MP10: PRPC020DAAN-RC, symbol Mechanical:Housing
- added MP11, MP12, MP14, MP16: generic, symbol Mechanical:Housing
- added MP13: 01020071Z, symbol Mechanical:Housing
- added MP9: Raspberry Pi Zero 2 W, symbol Mechanical:Housing
- H1, H2, H3, H4: footprint MountingHole:MountingHole_4mm -> MountingHole:MountingHole_3.2mm_M3
- MP1: Manufacturer custom (die-cut to drawing, TBD) -> custom (die-cut and folded to drawing, TBD)
- MP2: value RACO 257 -> NS1086; MPN RACO 257 -> NS1086; Manufacturer Hubbell RACO -> ABB (Carlon) Circuit Safe
- MP3: value RACO 250 -> JP108P; MPN RACO 250 -> JP108P; Manufacturer Hubbell RACO -> ABB (Carlon)
- MP4: value RACO 832 -> BH353A; MPN RACO 832 -> BH353A; Manufacturer Hubbell RACO -> ABB (Carlon) Superblue
- MP5, MP6, MP7: value LCBS-8-19 -> TR5252; MPN LCBS-8-19 -> TR5252; Manufacturer Essentra Components (Richco) -> Legrand Pass & Seymour
- MP8: value LCBS-8-19 -> generic; MPN LCBS-8-19 -> (none); Manufacturer Essentra Components (Richco) -> generic
Other:
- title: Mounting holes, SELV cover and box parts (BOM only) -> Holes; partition; enclosures, receptacles, Pi and hardware (BOM only)
- moved on the sheet: MP1, MP2, MP3, MP4, MP5, MP6, MP7, MP8

Commit message: designs/rpi-mains-relay: work-in-progress rework (6 receptacles, Pi Zero 2 W inside)
Co-Authored-By: Claude Opus 5.5 <noreply@anthropic.com>
Claude-Session: https://claude.ai/code/session_01VFJn9VbX8h27kf4LpLwEtn
Parts:
- removed MP16: generic, symbol Mechanical:Housing
- added MP15: generic, symbol Mechanical:Housing
Changed lines of the file:
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@@
 		(rev "A")
 		(company "kaesynth")
-		(comment 1 "H1-H6 board standoffs, H7-H10 Pi standoffs; MP1 partition; MP2-MP18 off-board items")
-		(comment 2 "RPi Zero 2 W six-outlet 120 VAC relay board (polycarbonate enclosure) — generated by kaesynth from design.py; do not edit by hand")
+		(comment 1 "H1-H6 board standoffs, H7-H10 Pi standoffs; MP1 partition; MP2-MP15 off-board items")
+		(comment 2 "RPi Zero 2 W 6-outlet 120 VAC relay board — generated by kaesynth from design.py; do not edit by hand")
 	)
 	(symbol
@@
 			)
 		)
-		(property "Description" "Partition: 1.5 mm polycarbonate UL 94 V-0 (Lexan FR class), full enclosure width, from the PCB surface to the lid, 10 mm folded foot; separates the field-wiring compartment from the PCB/Pi"
+		(property "Description" "Partition: 1.5 mm polycarbonate UL 94 V-0 (Lexan FR class): wall across the enclosure from the PCB to the lid at the J1-J4 south faces, plus a flat sheet die-cut around J1-J4 covering the PCB north of the wall; separates field wiring from the PCB/Pi"
 			(at 185.42 33.02 0)
 			(hide yes)
@@
 		(on_board no)
 		(dnp no)
-		(property "Reference" "MP16"
+		(property "Reference" "MP15"
 			(at 252.73 55.88 0)
 			(effects
@@
 			(project "rpi-mains-relay"
 				(path "/a30cabb5-b934-5e97-9aeb-aaefec3ba07a/3d33b6f9-21ed-5bfc-a356-a4c53021f7fa"
-					(reference "MP16")
-					(unit 1)
-				)
+					(reference "MP15")
+					(unit 1)
+				)

Commit message: designs/rpi-mains-relay: revision 3 — one enclosure (user decision)
User chose one enclosure (2026-10-23, Q-8). An ABB/Carlon NS14126 polycarbonate UL 50
Type 4X enclosure (14 x 12 x 6 in; Wi-Fi passes) holds the unchanged 200 x 150 mm board on
its back panel; three split-tab TR duplex receptacles mount in a 3-gang cut-out in the
cover on a 6.4 mm polycarbonate subplate, yokes bonded by pigtails, 14 AWG leads with a
service loop to J2-J4. A partition keeps receptacles and field wiring away from the board's
SELV side; the Pi is >= 150 mm from them. 15.5 W gives 49 C inside at a 40 C room.

No listed nonmetallic enclosure with receptacle openings in its cover was found, so
cover-mounted receptacles need a field evaluation or a UL 508A shop: new blocking Q-17.
All mains barriers ac=True. Build: 0 errors, 0 warnings, 31 waived, ERC clean, netlist
identical (L_IN now correctly flagged: relays sit on the wire side of the supply fuse;
the branch-breaker waiver covers it).

Co-Authored-By: Claude Opus 5.5 <noreply@anthropic.com>
Claude-Session: https://claude.ai/code/session_01VFJn9VbX8h27kf4LpLwEtn
Parts:
- MP2: value NS1086 -> NS14126; MPN NS1086 -> NS14126
- MP3: value JP108P -> JP1412P; MPN JP108P -> JP1412P
- MP4: value BH353A -> KAE-RPMR-MP4; MPN BH353A -> KAE-RPMR-MP4; Manufacturer ABB (Carlon) Superblue -> custom (machined to drawing, TBD)
Changed lines of the file:
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@@
 			)
 		)
-		(property "Value" "NS1086"
+		(property "Value" "NS14126"
 			(at 212.09 34.925 0)
 			(effects
@@
 			)
 		)
-		(property "Description" "Enclosure 10 x 8 x 6 in, polycarbonate, opaque screw cover, captive screws, nonmetallic hinges/rails; UL 50 / CSA C22.2 No.94.1 Types 4X, 12, 13 (file E88685); RF-transparent"
+		(property "Description" "Enclosure 14 x 12 x 6 in, polycarbonate, opaque screw cover, captive screws, nonmetallic hinges/rails; UL 50 / CSA C22.2 No.94.1 Types 4X, 12, 13 (file E88685); RF-transparent. The receptacle opening is cut in the cover (see MP4)"
 			(at 208.28 33.02 0)
 			(hide yes)
@@
 			)
 		)
-		(property "MPN" "NS1086"
+		(property "MPN" "NS14126"
 			(at 208.28 33.02 0)
 			(hide yes)
@@
 			)
 		)
-		(property "Value" "JP108P"
+		(property "Value" "JP1412P"
 			(at 232.41 34.925 0)
 			(effects
@@
 			)
 		)
-		(property "Description" "Back panel PVC 8.75 x 6.88 in for NS108x (10-32 x 3/8 screws ordered separately)"
+		(property "Description" "Back panel PVC 12.75 x 10.88 in for NS1412x (10-32 x 3/8 screws ordered separately)"
 			(at 228.6 33.02 0)
 			(hide yes)
@@
 			)
 		)
-		(property "MPN" "JP108P"
+		(property "MPN" "JP1412P"
 			(at 228.6 33.02 0)
 			(hide yes)
@@
 			)
 		)
-		(property "Value" "BH353A"
+		(property "Value" "KAE-RPMR-MP4"
 			(at 255.27 34.925 0)
 			(effects
@@
 			)
 		)
-		(property "Datasheet" "https://www.elliottelectric.com/P/Item/TAB/BH353A/"
+		(property "Datasheet" ""
 			(at 251.46 33.02 0)
 			(hide yes)
@@
 			)
 		)
-		(property "Description" "3-gang nonmetallic (PVC) device box, 53 in3, nail/screw mount, UL listed E11461"
+		(property "Description" "Receptacle subplate: 6.4 mm (1/4 in) polycarbonate UL 94 V-0, behind the cover's 3-gang cut-out, fixed to the cover with 6 nylon-insulated through bolts; 6-32 tapped at standard device-yoke spacing (3-9/32 in screw centres, 1-13/16 in gang pitch) for three duplex receptacles; the nylon 3-gang wallplate (MP8) clamps the cover from outside"
 			(at 251.46 33.02 0)
 			(hide yes)
@@
 			)
 		)
-		(property "MPN" "BH353A"
+		(property "MPN" "KAE-RPMR-MP4"
 			(at 251.46 33.02 0)
 			(hide yes)
@@
 			)
 		)
-		(property "Manufacturer" "ABB (Carlon) Superblue"
+		(property "Manufacturer" "custom (machined to drawing, TBD)"
 			(at 251.46 33.02 0)
 			(hide yes)
@@
 			)
 		)
-		(property "Description" "Field-wiring kit: 4 x listed nonmetallic NM-B cable connectors (1/2 in); 1 x listed 5-port lever splicing connector for the EGCs (e.g. WAGO 221-415); 3 x 14/3 NM-B with ground, ~0.5 m (E1 to E2); 3 x 6 in green EGC pigtails; 4 adhesive-free screw-on cable-tie mounts"
+		(property "Description" "Field-wiring kit: 1 x listed nonmetallic NM-B cable connector (1/2 in) for the branch; 1 x listed 5-port lever splicing connector for the EGCs (e.g. WAGO 221-415); receptacle leads 14 AWG THHN/THWN-2 Cu 600 V, 9 x 0.45 m (black/red/white per receptacle) with a 300 mm service loop for cover removal; 3 x green 14 AWG EGC pigtails; screw-on cable-tie mounts and a spiral wrap for the lead bundle"
 			(at 248.92 55.88 0)
 			(hide yes)

Commit message: designs/rpi-mains-relay: fix the revision-3 re-review findings
- Watchdog: turn-off back to <= 0.5 s (no source asked for faster); R21 1 M, C6 220 nF
  give a 150-340 ms window. wdsim.py (a time-domain model used by design.py's calcs):
  stuck high/low off in 165-356 ms, heartbeat gaps up to 152 ms ride through, chatter
  only at 2.9-6.7 Hz; heartbeat >= 20 Hz from a priority thread; test plan corrected.
- Finger-safe polycarbonate shield over the supply fuse, relay contacts, supply AC pins
  and line copper; receptacle backs shrouded.
- Cover receptacles: brass threaded inserts, fine-stranded 14 AWG leads with ferrules and
  strain relief, 20 N pull test; the field cut drops the enclosure to Type 1 (indoor dry),
  stated in Q-17.
- Minors fixed or answered. Build: 0 errors, ERC clean, netlist identical, 31 waived.

Co-Authored-By: Claude Opus 5.5 <noreply@anthropic.com>
Claude-Session: https://claude.ai/code/session_01VFJn9VbX8h27kf4LpLwEtn
Parts:
- added MP16: KAE-RPMR-MP16, symbol Mechanical:Housing
Changed lines of the file:
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@@
 			)
 		)
-		(property "Description" "Receptacle subplate: 6.4 mm (1/4 in) polycarbonate UL 94 V-0, behind the cover's 3-gang cut-out, fixed to the cover with 6 nylon-insulated through bolts; 6-32 tapped at standard device-yoke spacing (3-9/32 in screw centres, 1-13/16 in gang pitch) for three duplex receptacles; the nylon 3-gang wallplate (MP8) clamps the cover from outside"
+		(property "Description" "Receptacle subplate assembly: 6.4 mm (1/4 in) polycarbonate UL 94 V-0 plate behind the cover's 3-gang cut-out, fixed with 6 nylon-insulated through bolts; brass heat-set 6-32 inserts at standard yoke spacing (3-9/32 in screw centres, 1-13/16 in gang pitch), never threads cut in the plastic; a 1.5 mm polycarbonate rear shroud closes over the receptacle backs (finger-safe with the cover off), the leads leave through a strain-relief grommet; the nylon 3-gang wallplate (MP8) clamps the cover"
 			(at 251.46 33.02 0)
 			(hide yes)
@@
 			)
 		)
-		(property "Description" "Field-wiring kit: 1 x listed nonmetallic NM-B cable connector (1/2 in) for the branch; 1 x listed 5-port lever splicing connector for the EGCs (e.g. WAGO 221-415); receptacle leads 14 AWG THHN/THWN-2 Cu 600 V, 9 x 0.45 m (black/red/white per receptacle) with a 300 mm service loop for cover removal; 3 x green 14 AWG EGC pigtails; screw-on cable-tie mounts and a spiral wrap for the lead bundle"
+		(property "Description" "Field-wiring kit: 1 x listed nonmetallic NM-B cable connector (1/2 in) for the branch; 1 x listed 5-port lever splicing connector for the EGCs (e.g. WAGO 221-415); receptacle leads 14 AWG UL 1015 600 V 105 C fine-stranded Cu (Class K), 9 x 0.45 m (black/red/white per receptacle) with a 300 mm service loop for cover removal, ferrules at the WAGO end; 3 x green 14 AWG stranded EGC pigtails; strain relief at both ends; screw-on cable-tie mounts and a spiral wrap for the lead bundle"
 			(at 248.92 55.88 0)
 			(hide yes)
@@
 					(unit 1)
 				)
+			)
+		)
+	)
+	(symbol
+		(lib_id "Mechanical:Housing")
+		(at 33.02 81.28 0)
+		(unit 1)
+		(exclude_from_sim no)
+		(in_bom yes)
+		(on_board no)
+		(dnp no)
+		(property "Reference" "MP16"
+			(at 36.83 81.28 0)
+			(effects
+				(font (size 1.27 1.27))
+				(justify left)
+			)
+		)
+		(property "Value" "KAE-RPMR-MP16"
+			(at 36.83 83.185 0)
+			(effects
+				(font (size 1.27 1.27))
+				(justify left)
+			)
+		)
+		(property "Footprint" ""
+			(at 33.02 81.28 0)
+			(hide yes)
+			(effects
+				(font (size 1.27 1.27))
+			)
+		)
+		(property "Datasheet" ""
+			(at 33.02 81.28 0)
+			(hide yes)
+			(effects
+				(font (size 1.27 1.27))
+			)
+		)
+		(property "Description" "Mains-area shield: 1.0 mm clear polycarbonate UL 94 V-0 tray over the board from the MP1 wall to the barrier band (F1 and its clips, relay contact pins, PS1 AC end, L/L_SW copper), 35 mm above the board, 4 mm perforations (IP2X: finger probe cannot pass), flanges screwed to the back panel beyond both board ends; leaves only the SELV/Pi zone open when the cover is off"
+			(at 33.02 81.28 0)
+			(hide yes)
+			(effects
+				(font (size 1.27 1.27))
+			)
+		)
+		(property "MPN" "KAE-RPMR-MP16"
+			(at 33.02 81.28 0)
+			(hide yes)
+			(effects
+				(font (size 1.27 1.27))
+			)
+		)
+		(property "Manufacturer" "custom (folded to drawing, TBD)"
+			(at 33.02 81.28 0)
+			(hide yes)
+			(effects
+				(font (size 1.27 1.27))
+			)
+		)
+		(property "Block" "mech"
+			(at 33.02 81.28 0)
+			(hide yes)
+			(effects
+				(font (size 1.27 1.27))
+			)
+		)
+		(property "Component Class" "mech"
+			(at 33.02 81.28 0)
+			(hide yes)
+			(effects
+				(font (size 1.27 1.27))
+			)
+		)
+		(instances
+			(project "rpi-mains-relay"
+				(path "/a30cabb5-b934-5e97-9aeb-aaefec3ba07a/3d33b6f9-21ed-5bfc-a356-a4c53021f7fa"
+					(reference "MP16")
+					(unit 1)
+				)
