File: designs/leadacid-balancer/out/input.kicad_sch (KiCad schematic)
At the start: 16 parts, among them J1 1757271

Commit message: designs: work-in-progress (review fixes under way)
Co-Authored-By: Claude Opus 5.5 <noreply@anthropic.com>
Claude-Session: https://claude.ai/code/session_01VFJn9VbX8h27kf4LpLwEtn
Parts:
- removed XC1, XC10, XC2, XC3, XC4, XC5, XC6, XC7, XC8, XC9: 01000056Z, symbol Mechanical:Housing
- added XH1, XH2, XH3, XH4, XH5: 3576, symbol Mechanical:Housing
- F1, F2, F3, F4, F5: value 4A -> 6A; footprint Fuse:Fuseholder_Clip-5x20mm_Littelfuse_100_Inline_P20.50x4.60mm_D1.30mm_Horizontal -> custom:Fuseholder_Keystone_3576_10x38mm; Breaking 1500A -> 10000A; I2t (none) -> 63A2s; MPN 0477004.MXP -> KLKD006.T; Rating 4A -> 6A
