File: designs/leadacid-balancer/out/ch1.kicad_sch (KiCad schematic)
At the start: 127 parts, among them Q101 CSD18543Q3A, Q102 CSD18543Q3A, Q103 CSD18543Q3A, Q104 CSD18543Q3A, Q105 MMBT3906, Q106 2N7002, Q107 MMBT3906, U101 UCC21520ADWR, U102 UCC21520ADWR, U103 CD4047BM96, U104 TPS7A1601DGNR, U105 TPS7A1601DGNR, U106 TPS70950DBVR, U107 REF35250, U108 TLV7044PWR, U109 74LVC1G02, U110 SFH617A-3

Commit message: designs: work-in-progress (review fixes under way)
Co-Authored-By: Claude Opus 5.5 <noreply@anthropic.com>
Claude-Session: https://claude.ai/code/session_01VFJn9VbX8h27kf4LpLwEtn
Parts:
- added C151: 4.7u, Capacitor_SMD:C_0805_2012Metric, symbol Device:C
- added C152: 100n, Capacitor_SMD:C_0603_1608Metric, symbol Device:C
- added C153, C154: 470n, Capacitor_SMD:C_0603_1608Metric, symbol Device:C
- added D105: BAS16W, Package_TO_SOT_SMD:SOT-323_SC-70, symbol Diode:BAS16W
- added JP102: EN, Connector_PinHeader_2.54mm:PinHeader_1x02_P2.54mm_Vertical, symbol Jumper:Jumper_2_Open
- added JS102: 60900213421, symbol Mechanical:Housing
- added R154, R155, R156, R157, R160, R161, R162, R163, R166, R167, R168, R169: 2M, Resistor_SMD:R_1206_3216Metric, symbol Device:R
- added R158, R159: 4.7, Resistor_SMD:R_0603_1608Metric, symbol Device:R
- added R164, R165: 1.62M, Resistor_SMD:R_1206_3216Metric, symbol Device:R
- added R170, R171: 1.7M, Resistor_SMD:R_1206_3216Metric, symbol Device:R
- added R172: 825, Resistor_SMD:R_0603_1608Metric, symbol Device:R
- added R173, R174, R175, R178, R179: 4.99M, Resistor_SMD:R_0603_1608Metric, symbol Device:R
- added R176: 100k, Resistor_SMD:R_0603_1608Metric, symbol Device:R
- added R177: 249k, Resistor_SMD:R_0603_1608Metric, symbol Device:R
- added unit 2 of U109
- added unit 3 of U109
- added U111: TLV7044PWR, Package_SO:TSSOP-14_4.4x5mm_P0.65mm, symbol kaesynth:TLV7044PWR
- C138: value 2.2u -> 4.7u; footprint Capacitor_SMD:C_0603_1608Metric -> Capacitor_SMD:C_0805_2012Metric; MPN GRM188R71C225KE11D -> GRM21BR71E475KA73L; Voltage 16V -> 25V
- R126, R127, R130, R131: value 4.99M -> 2M; footprint Resistor_SMD:R_0603_1608Metric -> Resistor_SMD:R_1206_3216Metric; MPN CRCW06034M99FKEA -> TNPW12062M00BEEA; Manufacturer Vishay Dale -> Vishay Draloric; Package 0603 -> 1206; TCR (none) -> 25 ppm/K; Tolerance 1% -> 0.1%
- R128, R129: value 1M -> 1.58M; footprint Resistor_SMD:R_0603_1608Metric -> Resistor_SMD:R_1206_3216Metric; MPN CRCW06031M00FKEA -> TNPW12061M58BEEA; Manufacturer Vishay Dale -> Vishay Draloric; Package 0603 -> 1206; TCR (none) -> 25 ppm/K; Tolerance 1% -> 0.1%
- R132, R133: value 1.1M -> 1.74M; footprint Resistor_SMD:R_0603_1608Metric -> Resistor_SMD:R_1206_3216Metric; MPN CRCW06031M10FKEA -> TNPW12061M74BEEA; Manufacturer Vishay Dale -> Vishay Draloric; Package 0603 -> 1206; TCR (none) -> 25 ppm/K; Tolerance 1% -> 0.1%
- R134, R135: value 2.26M -> 2M; footprint Resistor_SMD:R_0603_1608Metric -> Resistor_SMD:R_1206_3216Metric; MPN CRCW06032M26FKEA -> TNPW12062M00BEEA; Manufacturer Vishay Dale -> Vishay Draloric; Package 0603 -> 1206; TCR (none) -> 25 ppm/K; Tolerance 1% -> 0.1%
- R136, R137: value 1M -> 1.85M; footprint Resistor_SMD:R_0603_1608Metric -> Resistor_SMD:R_1206_3216Metric; MPN CRCW06031M00FKEA -> TNPW12061M85BEEA; Manufacturer Vishay Dale -> Vishay Draloric; Package 0603 -> 1206; TCR (none) -> 25 ppm/K; Tolerance 1% -> 0.1%
- R142: value 100k -> 10k; MPN CRCW0603100KFKEA -> CRCW060310K0FKEA
- R145: value 249 -> 750; MPN CRCW0603249RFKEA -> CRCW0603750RFKEA
- U109: value 74LVC1G02 -> 74LVC2G02; footprint Package_TO_SOT_SMD:SOT-23-5 -> Package_SO:SSOP-8_2.95x2.8mm_P0.65mm; symbol 74xGxx:74LVC1G02 -> 74xGxx:74LVC2G02; MPN SN74LVC1G02DBVR -> SN74LVC2G02DCTR
Connections:
- net CH1_12VL: now also R159.1; no longer D102.1 (A)
- net CH1_12VU: now also R158.1; no longer D101.1 (A)
- net CH1_FLT: now also U109.7, U109.6; no longer Q105.3 (C), R144.1, R145.1, U109.2
- net CH1_FLT_N: now also U109.1, U109.2
- net CH1_N: now also U111.5 (INB+), U111.9 (INC-)
- net CH1_NCHG: now also U109.5; no longer U109.1
- net CH1_PHI: now also R157.2; no longer R131.2
- net CH1_PLO: now also R155.2; no longer R127.2
- net CH1_RUN: now also R172.1, R176.1, U109.3; no longer U109.4
- net CH1_V5: now also C152.1, R173.1, U109.8 (VCC), U111.4 (VCC); no longer U109.5 (VCC)
- net CH1_VREF: now also U111.2 (INA-)
- net TAP0: now also D103.1 (K), C151.2, C152.2, C153.2, C154.2, R164.2, R165.2, R170.2, R171.2, R174.2, U109.4 (GND), U111.11 (VEE), U111.3 (INA+); no longer U101.5 (DIS), U102.5 (DIS), U109.3 (GND)
- net TAP2: now also R160.1, R166.1
- net ALM_C renamed ALM_S1
- net ALM_S1: now also JP102.1 (A)
- net ALM_E renamed ALM_S2
- net ALM_S2: now also JP102.2 (B)
- net CH1_N_M renamed CH1_N_M1
- net CH1_OPTO_A renamed CH1_OKA
- net CH1_OKA: now also R172.2, U111.7 (OUTB), U111.8 (OUTC); no longer D103.1 (K)
- net CH1_PHI_M renamed CH1_PHI_M1
- net CH1_PLO_M renamed CH1_PLO_M1
- net CH1_PON_A renamed CH1_PON_M1
- net CH1_PON_B renamed CH1_PON_M2
- net CH1_PON_C renamed CH1_PON_M3
- new net CH1_BSL_A: D102.1 (A), R159.2
- new net CH1_BSU_A: D101.1 (A), R158.2
- new net CH1_LEDQ: Q105.3 (C), R144.1, R145.1
- new net CH1_PAUSE: D105.1 (A), R175.1, R176.2, R178.1, U101.5 (DIS), U102.5 (DIS), U111.14 (OUTD)
- new net CH1_PDA: D105.3 (K), R177.1
- new net CH1_PHI_M2: R131.2, R156.1
- new net CH1_PHI_M3: R156.2, R157.1
- new net CH1_PLO_M2: R127.2, R154.1
- new net CH1_PLO_M3: R154.2, R155.1
- new net CH1_PWH: C153.1, R163.2, R164.1, R165.1, U111.6 (INB-)
- new net CH1_PWH_M1: R160.2, R161.1
- new net CH1_PWH_M2: R161.2, R162.1
- new net CH1_PWH_M3: R162.2, R163.1
- new net CH1_PWL: C154.1, R169.2, R170.1, R171.1, U111.10 (INC+)
- new net CH1_PWL_M1: R166.2, R167.1
- new net CH1_PWL_M2: R167.2, R168.1
- new net CH1_PWL_M3: R168.2, R169.1
- new net CH1_TCT: C151.1, R177.2, R179.2, U111.13 (IND-)
- new net CH1_TPN: R173.2, R174.1, R175.2, U111.12 (IND+)
- new net CH1_TSM: R178.2, R179.1
- no-connect marks 17 -> 19
Other:
- moved on the sheet: C101, C102, C103, C104, C105, C106, C107, C108, C109, C110, C111, C112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

Commit message: designs: work-in-progress (review fixes under way)
Co-Authored-By: Claude Opus 5.5 <noreply@anthropic.com>
Claude-Session: https://claude.ai/code/session_01VFJn9VbX8h27kf4LpLwEtn
Parts:
- removed R164, R165: 1.62M, Resistor_SMD:R_1206_3216Metric, symbol Device:R
- removed R166, R167, R168, R169: 2M, Resistor_SMD:R_1206_3216Metric, symbol Device:R
- removed R170, R171: 1.7M, Resistor_SMD:R_1206_3216Metric, symbol Device:R
- R132, R133: value 1.74M -> 1.7M; MPN TNPW12061M74BEEA -> TNPW12061M70BEEA
- R155: value 2M -> 1.96M; MPN TNPW12062M00BEEA -> TNPW12061M96BEEA
- R160, R161: value 2M -> 30.9k; footprint Resistor_SMD:R_1206_3216Metric -> Resistor_SMD:R_0603_1608Metric; MPN TNPW12062M00BEEA -> CRCW060330K9FKEA; Manufacturer Vishay Draloric -> Vishay Dale; Package 1206 -> 0603; TCR 25 ppm/K -> (none); Tolerance 0.1% -> 1%
- R162, R163: value 2M -> 36.5k; footprint Resistor_SMD:R_1206_3216Metric -> Resistor_SMD:R_0603_1608Metric; MPN TNPW12062M00BEEA -> CRCW060336K5FKEA; Manufacturer Vishay Draloric -> Vishay Dale; Package 1206 -> 0603; TCR 25 ppm/K -> (none); Tolerance 0.1% -> 1%
Connections:
- net CH1_PHI: now also R162.1, R163.1; no longer R132.1, R133.1
- net CH1_PLO: now also R160.2, R161.2; no longer R155.2
- net CH1_PWH: now also R155.2, R160.1, R161.1; no longer R163.2
- net CH1_PWL: now also R132.1, R133.1, R162.2, R163.2
- net TAP2: no longer R160.1
- removed net CH1_PWH_M1: R160.2, R161.1
- removed net CH1_PWH_M2: R161.2, R162.1
- removed net CH1_PWH_M3: R162.2, R163.1
Other:
- moved on the sheet: C101, C102, C103, C104, C105, C106, C107, C108, C109, C118, C126, C127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

Commit message: designs/leadacid-balancer: fix the independent review's blocker and majors
- B-1: board fuse KLKD006.T (6 A, 600 VDC, 10 kA DC, 63 A2s) in Keystone 3576 holders
  (custom footprint; board 180 x 130 mm); worst board fault 670 A vs 10 kA.
- M-1: 0.1 % thin-film supervisor strings; tolerance incl. comparator offset, half
  hysteresis and TCR is +/-1.34 % vs the 1.5 % budget; worst-case trip points in calcs.
- M-2: RUN = NOR(NCHG, FLT) on a logic gate; the fault transistor only drives the LED.
- M-3: +/-4 % imbalance warning opens the alarm; silent current into a failing battery
  <= 2.44 A (was 4.4 A).
- M-4: fail-safe alarm loop (closed only while all channels are healthy); periodic tap
  check catches a floating tap in 1.14 s.
- Minors fixed or answered. Build: 0 errors, ERC clean, netlist identical, 31 waived;
  N = 2/3 variants clean.

Co-Authored-By: Claude Opus 5.5 <noreply@anthropic.com>
Claude-Session: https://claude.ai/code/session_01VFJn9VbX8h27kf4LpLwEtn
Parts:
- R158, R159: value 4.7 -> 10; MPN CRCW06034R70FKEA -> CRCW060310R0FKEA
- R160, R161: footprint Resistor_SMD:R_0603_1608Metric -> Resistor_SMD:R_1206_3216Metric; MPN CRCW060330K9FKEA -> TNPW120630K9BEEA; Manufacturer Vishay Dale -> Vishay Draloric; Package 0603 -> 1206; TCR (none) -> 25 ppm/K; Tolerance 1% -> 0.1%
- R162, R163: footprint Resistor_SMD:R_0603_1608Metric -> Resistor_SMD:R_1206_3216Metric; MPN CRCW060336K5FKEA -> TNPW120636K5BEEA; Manufacturer Vishay Dale -> Vishay Draloric; Package 0603 -> 1206; TCR (none) -> 25 ppm/K; Tolerance 1% -> 0.1%
Changed lines of the file:
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@@
 			)
 		)
-		(property "Value" "4.7"
+		(property "Value" "10"
 			(at 370.84 180.34 90)
 			(effects
@@
 			)
 		)
-		(property "Description" "Resistor 4.7 1% 0603"
+		(property "Description" "Resistor 10 1% 0603"
 			(at 370.84 180.34 0)
 			(hide yes)
@@
 			)
 		)
-		(property "MPN" "CRCW06034R70FKEA"
+		(property "MPN" "CRCW060310R0FKEA"
 			(at 370.84 180.34 0)
 			(hide yes)
@@
 			)
 		)
-		(property "Value" "4.7"
+		(property "Value" "10"
 			(at 381 180.34 90)
 			(effects
@@
 			)
 		)
-		(property "Description" "Resistor 4.7 1% 0603"
+		(property "Description" "Resistor 10 1% 0603"
 			(at 381 180.34 0)
 			(hide yes)
@@
 			)
 		)
-		(property "MPN" "CRCW06034R70FKEA"
+		(property "MPN" "CRCW060310R0FKEA"
 			(at 381 180.34 0)
 			(hide yes)
@@
 			)
 		)
-		(property "Footprint" "Resistor_SMD:R_0603_1608Metric"
+		(property "Footprint" "Resistor_SMD:R_1206_3216Metric"
 			(at 73.66 322.58 0)
 			(hide yes)
@@
 			)
 		)
-		(property "Datasheet" "https://www.vishay.com/docs/20035/dcrcwe3.pdf"
+		(property "Datasheet" "https://www.vishay.com/docs/28758/tnpw_e3.pdf"
 			(at 73.66 322.58 0)
 			(hide yes)
@@
 			)
 		)
-		(property "Description" "Resistor 30.9k 1% 0603"
+		(property "Description" "Resistor 30.9k 0.1% 1206"
 			(at 73.66 322.58 0)
 			(hide yes)
@@
 			)
 		)
-		(property "MPN" "CRCW060330K9FKEA"
+		(property "MPN" "TNPW120630K9BEEA"
 			(at 73.66 322.58 0)
 			(hide yes)
@@
 			)
 		)
-		(property "Manufacturer" "Vishay Dale"
+		(property "Manufacturer" "Vishay Draloric"
 			(at 73.66 322.58 0)
 			(hide yes)
@@
 			)
 		)
-		(property "Tolerance" "1%"
+		(property "Tolerance" "0.1%"
 			(at 73.66 322.58 0)
 			(hide yes)
@@
 			)
 		)
-		(property "Package" "0603"
+		(property "Package" "1206"
+			(at 73.66 322.58 0)
+			(hide yes)
+			(effects
+				(font (size 1.27 1.27))
+			)
+		)
+		(property "TCR" "25 ppm/K"
 			(at 73.66 322.58 0)
 			(hide yes)
@@
 			)
 		)
-		(property "Footprint" "Resistor_SMD:R_0603_1608Metric"
+		(property "Footprint" "Resistor_SMD:R_1206_3216Metric"
 			(at 86.36 322.58 0)
 			(hide yes)
@@
 			)
 		)
-		(property "Datasheet" "https://www.vishay.com/docs/20035/dcrcwe3.pdf"
+		(property "Datasheet" "https://www.vishay.com/docs/28758/tnpw_e3.pdf"
 			(at 86.36 322.58 0)
 			(hide yes)
@@
 			)
 		)
-		(property "Description" "Resistor 30.9k 1% 0603"
+		(property "Description" "Resistor 30.9k 0.1% 1206"
 			(at 86.36 322.58 0)
 			(hide yes)
@@
 			)
 		)
-		(property "MPN" "CRCW060330K9FKEA"
+		(property "MPN" "TNPW120630K9BEEA"
 			(at 86.36 322.58 0)
 			(hide yes)
@@
 			)
 		)
-		(property "Manufacturer" "Vishay Dale"
+		(property "Manufacturer" "Vishay Draloric"
 			(at 86.36 322.58 0)
 			(hide yes)
@@
 			)
 		)
-		(property "Tolerance" "1%"
+		(property "Tolerance" "0.1%"
 			(at 86.36 322.58 0)
 			(hide yes)
@@
 			)
 		)
-		(property "Package" "0603"
+		(property "Package" "1206"
+			(at 86.36 322.58 0)
+			(hide yes)
+			(effects
+				(font (size 1.27 1.27))
+			)
+		)
+		(property "TCR" "25 ppm/K"
 			(at 86.36 322.58 0)
 			(hide yes)
@@
 			)
 		)
-		(property "Footprint" "Resistor_SMD:R_0603_1608Metric"
+		(property "Footprint" "Resistor_SMD:R_1206_3216Metric"
 			(at 40.64 375.92 0)
 			(hide yes)
@@
 			)
 		)
-		(property "Datasheet" "https://www.vishay.com/docs/20035/dcrcwe3.pdf"
+		(property "Datasheet" "https://www.vishay.com/docs/28758/tnpw_e3.pdf"
 			(at 40.64 375.92 0)
 			(hide yes)
@@
 			)
 		)
-		(property "Description" "Resistor 36.5k 1% 0603"
+		(property "Description" "Resistor 36.5k 0.1% 1206"
 			(at 40.64 375.92 0)
 			(hide yes)
@@
 			)
 		)
-		(property "MPN" "CRCW060336K5FKEA"
+		(property "MPN" "TNPW120636K5BEEA"
 			(at 40.64 375.92 0)
 			(hide yes)
@@
 			)
 		)
-		(property "Manufacturer" "Vishay Dale"
+		(property "Manufacturer" "Vishay Draloric"
 			(at 40.64 375.92 0)
 			(hide yes)
@@
 			)
 		)
-		(property "Tolerance" "1%"
+		(property "Tolerance" "0.1%"
 			(at 40.64 375.92 0)
 			(hide yes)
@@
 			)
 		)
-		(property "Package" "0603"
+		(property "Package" "1206"
+			(at 40.64 375.92 0)
+			(hide yes)
+			(effects
+				(font (size 1.27 1.27))
+			)
+		)
+		(property "TCR" "25 ppm/K"
 			(at 40.64 375.92 0)
 			(hide yes)
@@
 			)
 		)
-		(property "Footprint" "Resistor_SMD:R_0603_1608Metric"
+		(property "Footprint" "Resistor_SMD:R_1206_3216Metric"
 			(at 50.8 375.92 0)
 			(hide yes)
@@
 			)
 		)
-		(property "Datasheet" "https://www.vishay.com/docs/20035/dcrcwe3.pdf"
+		(property "Datasheet" "https://www.vishay.com/docs/28758/tnpw_e3.pdf"
 			(at 50.8 375.92 0)
 			(hide yes)
@@
 			)
 		)
-		(property "Description" "Resistor 36.5k 1% 0603"
+		(property "Description" "Resistor 36.5k 0.1% 1206"
 			(at 50.8 375.92 0)
 			(hide yes)
@@
 			)
 		)
-		(property "MPN" "CRCW060336K5FKEA"
+		(property "MPN" "TNPW120636K5BEEA"
 			(at 50.8 375.92 0)
 			(hide yes)
@@
 			)
 		)
-		(property "Manufacturer" "Vishay Dale"
+		(property "Manufacturer" "Vishay Draloric"
 			(at 50.8 375.92 0)
 			(hide yes)
@@
 			)
 		)
-		(property "Tolerance" "1%"
+		(property "Tolerance" "0.1%"
 			(at 50.8 375.92 0)
 			(hide yes)
@@
 			)
 		)
-		(property "Package" "0603"
+		(property "Package" "1206"
+			(at 50.8 375.92 0)
+			(hide yes)
+			(effects
+				(font (size 1.27 1.27))
+			)
+		)
+		(property "TCR" "25 ppm/K"
 			(at 50.8 375.92 0)
 			(hide yes)
