File: designs/leadacid-balancer/out/ch2.kicad_sch (KiCad schematic)
At the start: 127 parts, among them Q201 CSD18543Q3A, Q202 CSD18543Q3A, Q203 CSD18543Q3A, Q204 CSD18543Q3A, Q205 MMBT3906, Q206 2N7002, Q207 MMBT3906, U201 UCC21520ADWR, U202 UCC21520ADWR, U203 CD4047BM96, U204 TPS7A1601DGNR, U205 TPS7A1601DGNR, U206 TPS70950DBVR, U207 REF35250, U208 TLV7044PWR, U209 74LVC1G02, U210 SFH617A-3

Commit message: designs: work-in-progress (review fixes under way)
Co-Authored-By: Claude Opus 5.5 <noreply@anthropic.com>
Claude-Session: https://claude.ai/code/session_01VFJn9VbX8h27kf4LpLwEtn
Parts:
- added C251: 4.7u, Capacitor_SMD:C_0805_2012Metric, symbol Device:C
- added C252: 100n, Capacitor_SMD:C_0603_1608Metric, symbol Device:C
- added C253, C254: 470n, Capacitor_SMD:C_0603_1608Metric, symbol Device:C
- added D205: BAS16W, Package_TO_SOT_SMD:SOT-323_SC-70, symbol Diode:BAS16W
- added JP202: EN, Connector_PinHeader_2.54mm:PinHeader_1x02_P2.54mm_Vertical, symbol Jumper:Jumper_2_Open
- added JS202: 60900213421, symbol Mechanical:Housing
- added R254, R255, R256, R257, R260, R261, R262, R263, R266, R267, R268, R269: 2M, Resistor_SMD:R_1206_3216Metric, symbol Device:R
- added R258, R259: 4.7, Resistor_SMD:R_0603_1608Metric, symbol Device:R
- added R264, R265: 1.62M, Resistor_SMD:R_1206_3216Metric, symbol Device:R
- added R270, R271: 1.7M, Resistor_SMD:R_1206_3216Metric, symbol Device:R
- added R272: 825, Resistor_SMD:R_0603_1608Metric, symbol Device:R
- added R273, R274, R275, R278, R279: 4.99M, Resistor_SMD:R_0603_1608Metric, symbol Device:R
- added R276: 100k, Resistor_SMD:R_0603_1608Metric, symbol Device:R
- added R277: 249k, Resistor_SMD:R_0603_1608Metric, symbol Device:R
- added unit 2 of U209
- added unit 3 of U209
- added U211: TLV7044PWR, Package_SO:TSSOP-14_4.4x5mm_P0.65mm, symbol kaesynth:TLV7044PWR
- C238: value 2.2u -> 4.7u; footprint Capacitor_SMD:C_0603_1608Metric -> Capacitor_SMD:C_0805_2012Metric; MPN GRM188R71C225KE11D -> GRM21BR71E475KA73L; Voltage 16V -> 25V
- R226, R227, R230, R231: value 4.99M -> 2M; footprint Resistor_SMD:R_0603_1608Metric -> Resistor_SMD:R_1206_3216Metric; MPN CRCW06034M99FKEA -> TNPW12062M00BEEA; Manufacturer Vishay Dale -> Vishay Draloric; Package 0603 -> 1206; TCR (none) -> 25 ppm/K; Tolerance 1% -> 0.1%
- R228, R229: value 1M -> 1.58M; footprint Resistor_SMD:R_0603_1608Metric -> Resistor_SMD:R_1206_3216Metric; MPN CRCW06031M00FKEA -> TNPW12061M58BEEA; Manufacturer Vishay Dale -> Vishay Draloric; Package 0603 -> 1206; TCR (none) -> 25 ppm/K; Tolerance 1% -> 0.1%
- R232, R233: value 1.1M -> 1.74M; footprint Resistor_SMD:R_0603_1608Metric -> Resistor_SMD:R_1206_3216Metric; MPN CRCW06031M10FKEA -> TNPW12061M74BEEA; Manufacturer Vishay Dale -> Vishay Draloric; Package 0603 -> 1206; TCR (none) -> 25 ppm/K; Tolerance 1% -> 0.1%
- R234, R235: value 2.26M -> 2M; footprint Resistor_SMD:R_0603_1608Metric -> Resistor_SMD:R_1206_3216Metric; MPN CRCW06032M26FKEA -> TNPW12062M00BEEA; Manufacturer Vishay Dale -> Vishay Draloric; Package 0603 -> 1206; TCR (none) -> 25 ppm/K; Tolerance 1% -> 0.1%
- R236, R237: value 1M -> 1.85M; footprint Resistor_SMD:R_0603_1608Metric -> Resistor_SMD:R_1206_3216Metric; MPN CRCW06031M00FKEA -> TNPW12061M85BEEA; Manufacturer Vishay Dale -> Vishay Draloric; Package 0603 -> 1206; TCR (none) -> 25 ppm/K; Tolerance 1% -> 0.1%
- R242: value 100k -> 10k; MPN CRCW0603100KFKEA -> CRCW060310K0FKEA
- R245: value 249 -> 750; MPN CRCW0603249RFKEA -> CRCW0603750RFKEA
- U209: value 74LVC1G02 -> 74LVC2G02; footprint Package_TO_SOT_SMD:SOT-23-5 -> Package_SO:SSOP-8_2.95x2.8mm_P0.65mm; symbol 74xGxx:74LVC1G02 -> 74xGxx:74LVC2G02; MPN SN74LVC1G02DBVR -> SN74LVC2G02DCTR
Connections:
- net CH2_12VL: now also R259.1; no longer D202.1 (A)
- net CH2_12VU: now also R258.1; no longer D201.1 (A)
- net CH2_FLT: now also U209.7, U209.6; no longer Q205.3 (C), R244.1, R245.1, U209.2
- net CH2_FLT_N: now also U209.1, U209.2
- net CH2_N: now also U211.5 (INB+), U211.9 (INC-)
- net CH2_NCHG: now also U209.5; no longer U209.1
- net CH2_PHI: now also R257.2; no longer R231.2
- net CH2_PLO: now also R255.2; no longer R227.2
- net CH2_RUN: now also R272.1, R276.1, U209.3; no longer U209.4
- net CH2_V5: now also C252.1, R273.1, U209.8 (VCC), U211.4 (VCC); no longer U209.5 (VCC)
- net CH2_VREF: now also U211.2 (INA-)
- net TAP1: now also D203.1 (K), C251.2, C252.2, C253.2, C254.2, R264.2, R265.2, R270.2, R271.2, R274.2, U209.4 (GND), U211.11 (VEE), U211.3 (INA+); no longer U201.5 (DIS), U202.5 (DIS), U209.3 (GND)
- net TAP3: now also R260.1, R266.1
- net ALM_C renamed ALM_S2
- net ALM_S2: now also JP202.1 (A)
- net ALM_E renamed ALM_S3
- net ALM_S3: now also JP202.2 (B)
- net CH2_N_M renamed CH2_N_M1
- net CH2_OPTO_A renamed CH2_OKA
- net CH2_OKA: now also R272.2, U211.7 (OUTB), U211.8 (OUTC); no longer D203.1 (K)
- net CH2_PHI_M renamed CH2_PHI_M1
- net CH2_PLO_M renamed CH2_PLO_M1
- net CH2_PON_A renamed CH2_PON_M1
- net CH2_PON_B renamed CH2_PON_M2
- net CH2_PON_C renamed CH2_PON_M3
- new net CH2_BSL_A: D202.1 (A), R259.2
- new net CH2_BSU_A: D201.1 (A), R258.2
- new net CH2_LEDQ: Q205.3 (C), R244.1, R245.1
- new net CH2_PAUSE: D205.1 (A), R275.1, R276.2, R278.1, U201.5 (DIS), U202.5 (DIS), U211.14 (OUTD)
- new net CH2_PDA: D205.3 (K), R277.1
- new net CH2_PHI_M2: R231.2, R256.1
- new net CH2_PHI_M3: R256.2, R257.1
- new net CH2_PLO_M2: R227.2, R254.1
- new net CH2_PLO_M3: R254.2, R255.1
- new net CH2_PWH: C253.1, R263.2, R264.1, R265.1, U211.6 (INB-)
- new net CH2_PWH_M1: R260.2, R261.1
- new net CH2_PWH_M2: R261.2, R262.1
- new net CH2_PWH_M3: R262.2, R263.1
- new net CH2_PWL: C254.1, R269.2, R270.1, R271.1, U211.10 (INC+)
- new net CH2_PWL_M1: R266.2, R267.1
- new net CH2_PWL_M2: R267.2, R268.1
- new net CH2_PWL_M3: R268.2, R269.1
- new net CH2_TCT: C251.1, R277.2, R279.2, U211.13 (IND-)
- new net CH2_TPN: R273.2, R274.1, R275.2, U211.12 (IND+)
- new net CH2_TSM: R278.2, R279.1
- no-connect marks 17 -> 19
Other:
- moved on the sheet: C201, C202, C203, C204, C205, C206, C207, C208, C209, C210, C211, C212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

Commit message: designs: work-in-progress (review fixes under way)
Co-Authored-By: Claude Opus 5.5 <noreply@anthropic.com>
Claude-Session: https://claude.ai/code/session_01VFJn9VbX8h27kf4LpLwEtn
Parts:
- removed R264, R265: 1.62M, Resistor_SMD:R_1206_3216Metric, symbol Device:R
- removed R266, R267, R268, R269: 2M, Resistor_SMD:R_1206_3216Metric, symbol Device:R
- removed R270, R271: 1.7M, Resistor_SMD:R_1206_3216Metric, symbol Device:R
- R232, R233: value 1.74M -> 1.7M; MPN TNPW12061M74BEEA -> TNPW12061M70BEEA
- R255: value 2M -> 1.96M; MPN TNPW12062M00BEEA -> TNPW12061M96BEEA
- R260, R261: value 2M -> 30.9k; footprint Resistor_SMD:R_1206_3216Metric -> Resistor_SMD:R_0603_1608Metric; MPN TNPW12062M00BEEA -> CRCW060330K9FKEA; Manufacturer Vishay Draloric -> Vishay Dale; Package 1206 -> 0603; TCR 25 ppm/K -> (none); Tolerance 0.1% -> 1%
- R262, R263: value 2M -> 36.5k; footprint Resistor_SMD:R_1206_3216Metric -> Resistor_SMD:R_0603_1608Metric; MPN TNPW12062M00BEEA -> CRCW060336K5FKEA; Manufacturer Vishay Draloric -> Vishay Dale; Package 1206 -> 0603; TCR 25 ppm/K -> (none); Tolerance 0.1% -> 1%
Connections:
- net CH2_PHI: now also R262.1, R263.1; no longer R232.1, R233.1
- net CH2_PLO: now also R260.2, R261.2; no longer R255.2
- net CH2_PWH: now also R255.2, R260.1, R261.1; no longer R263.2
- net CH2_PWL: now also R232.1, R233.1, R262.2, R263.2
- net TAP3: no longer R260.1
- removed net CH2_PWH_M1: R260.2, R261.1
- removed net CH2_PWH_M2: R261.2, R262.1
- removed net CH2_PWH_M3: R262.2, R263.1
Other:
- moved on the sheet: C201, C202, C203, C204, C205, C206, C207, C208, C209, C218, C226, C227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

Commit message: designs/leadacid-balancer: fix the independent review's blocker and majors
- B-1: board fuse KLKD006.T (6 A, 600 VDC, 10 kA DC, 63 A2s) in Keystone 3576 holders
  (custom footprint; board 180 x 130 mm); worst board fault 670 A vs 10 kA.
- M-1: 0.1 % thin-film supervisor strings; tolerance incl. comparator offset, half
  hysteresis and TCR is +/-1.34 % vs the 1.5 % budget; worst-case trip points in calcs.
- M-2: RUN = NOR(NCHG, FLT) on a logic gate; the fault transistor only drives the LED.
- M-3: +/-4 % imbalance warning opens the alarm; silent current into a failing battery
  <= 2.44 A (was 4.4 A).
- M-4: fail-safe alarm loop (closed only while all channels are healthy); periodic tap
  check catches a floating tap in 1.14 s.
- Minors fixed or answered. Build: 0 errors, ERC clean, netlist identical, 31 waived;
  N = 2/3 variants clean.

Co-Authored-By: Claude Opus 5.5 <noreply@anthropic.com>
Claude-Session: https://claude.ai/code/session_01VFJn9VbX8h27kf4LpLwEtn
Parts:
- R258, R259: value 4.7 -> 10; MPN CRCW06034R70FKEA -> CRCW060310R0FKEA
- R260, R261: footprint Resistor_SMD:R_0603_1608Metric -> Resistor_SMD:R_1206_3216Metric; MPN CRCW060330K9FKEA -> TNPW120630K9BEEA; Manufacturer Vishay Dale -> Vishay Draloric; Package 0603 -> 1206; TCR (none) -> 25 ppm/K; Tolerance 1% -> 0.1%
- R262, R263: footprint Resistor_SMD:R_0603_1608Metric -> Resistor_SMD:R_1206_3216Metric; MPN CRCW060336K5FKEA -> TNPW120636K5BEEA; Manufacturer Vishay Dale -> Vishay Draloric; Package 0603 -> 1206; TCR (none) -> 25 ppm/K; Tolerance 1% -> 0.1%
Changed lines of the file:
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@@
 			)
 		)
-		(property "Value" "4.7"
+		(property "Value" "10"
 			(at 370.84 180.34 90)
 			(effects
@@
 			)
 		)
-		(property "Description" "Resistor 4.7 1% 0603"
+		(property "Description" "Resistor 10 1% 0603"
 			(at 370.84 180.34 0)
 			(hide yes)
@@
 			)
 		)
-		(property "MPN" "CRCW06034R70FKEA"
+		(property "MPN" "CRCW060310R0FKEA"
 			(at 370.84 180.34 0)
 			(hide yes)
@@
 			)
 		)
-		(property "Value" "4.7"
+		(property "Value" "10"
 			(at 381 180.34 90)
 			(effects
@@
 			)
 		)
-		(property "Description" "Resistor 4.7 1% 0603"
+		(property "Description" "Resistor 10 1% 0603"
 			(at 381 180.34 0)
 			(hide yes)
@@
 			)
 		)
-		(property "MPN" "CRCW06034R70FKEA"
+		(property "MPN" "CRCW060310R0FKEA"
 			(at 381 180.34 0)
 			(hide yes)
@@
 			)
 		)
-		(property "Footprint" "Resistor_SMD:R_0603_1608Metric"
+		(property "Footprint" "Resistor_SMD:R_1206_3216Metric"
 			(at 73.66 322.58 0)
 			(hide yes)
@@
 			)
 		)
-		(property "Datasheet" "https://www.vishay.com/docs/20035/dcrcwe3.pdf"
+		(property "Datasheet" "https://www.vishay.com/docs/28758/tnpw_e3.pdf"
 			(at 73.66 322.58 0)
 			(hide yes)
@@
 			)
 		)
-		(property "Description" "Resistor 30.9k 1% 0603"
+		(property "Description" "Resistor 30.9k 0.1% 1206"
 			(at 73.66 322.58 0)
 			(hide yes)
@@
 			)
 		)
-		(property "MPN" "CRCW060330K9FKEA"
+		(property "MPN" "TNPW120630K9BEEA"
 			(at 73.66 322.58 0)
 			(hide yes)
@@
 			)
 		)
-		(property "Manufacturer" "Vishay Dale"
+		(property "Manufacturer" "Vishay Draloric"
 			(at 73.66 322.58 0)
 			(hide yes)
@@
 			)
 		)
-		(property "Tolerance" "1%"
+		(property "Tolerance" "0.1%"
 			(at 73.66 322.58 0)
 			(hide yes)
@@
 			)
 		)
-		(property "Package" "0603"
+		(property "Package" "1206"
+			(at 73.66 322.58 0)
+			(hide yes)
+			(effects
+				(font (size 1.27 1.27))
+			)
+		)
+		(property "TCR" "25 ppm/K"
 			(at 73.66 322.58 0)
 			(hide yes)
@@
 			)
 		)
-		(property "Footprint" "Resistor_SMD:R_0603_1608Metric"
+		(property "Footprint" "Resistor_SMD:R_1206_3216Metric"
 			(at 86.36 322.58 0)
 			(hide yes)
@@
 			)
 		)
-		(property "Datasheet" "https://www.vishay.com/docs/20035/dcrcwe3.pdf"
+		(property "Datasheet" "https://www.vishay.com/docs/28758/tnpw_e3.pdf"
 			(at 86.36 322.58 0)
 			(hide yes)
@@
 			)
 		)
-		(property "Description" "Resistor 30.9k 1% 0603"
+		(property "Description" "Resistor 30.9k 0.1% 1206"
 			(at 86.36 322.58 0)
 			(hide yes)
@@
 			)
 		)
-		(property "MPN" "CRCW060330K9FKEA"
+		(property "MPN" "TNPW120630K9BEEA"
 			(at 86.36 322.58 0)
 			(hide yes)
@@
 			)
 		)
-		(property "Manufacturer" "Vishay Dale"
+		(property "Manufacturer" "Vishay Draloric"
 			(at 86.36 322.58 0)
 			(hide yes)
@@
 			)
 		)
-		(property "Tolerance" "1%"
+		(property "Tolerance" "0.1%"
 			(at 86.36 322.58 0)
 			(hide yes)
@@
 			)
 		)
-		(property "Package" "0603"
+		(property "Package" "1206"
+			(at 86.36 322.58 0)
+			(hide yes)
+			(effects
+				(font (size 1.27 1.27))
+			)
+		)
+		(property "TCR" "25 ppm/K"
 			(at 86.36 322.58 0)
 			(hide yes)
@@
 			)
 		)
-		(property "Footprint" "Resistor_SMD:R_0603_1608Metric"
+		(property "Footprint" "Resistor_SMD:R_1206_3216Metric"
 			(at 40.64 375.92 0)
 			(hide yes)
@@
 			)
 		)
-		(property "Datasheet" "https://www.vishay.com/docs/20035/dcrcwe3.pdf"
+		(property "Datasheet" "https://www.vishay.com/docs/28758/tnpw_e3.pdf"
 			(at 40.64 375.92 0)
 			(hide yes)
@@
 			)
 		)
-		(property "Description" "Resistor 36.5k 1% 0603"
+		(property "Description" "Resistor 36.5k 0.1% 1206"
 			(at 40.64 375.92 0)
 			(hide yes)
@@
 			)
 		)
-		(property "MPN" "CRCW060336K5FKEA"
+		(property "MPN" "TNPW120636K5BEEA"
 			(at 40.64 375.92 0)
 			(hide yes)
@@
 			)
 		)
-		(property "Manufacturer" "Vishay Dale"
+		(property "Manufacturer" "Vishay Draloric"
 			(at 40.64 375.92 0)
 			(hide yes)
@@
 			)
 		)
-		(property "Tolerance" "1%"
+		(property "Tolerance" "0.1%"
 			(at 40.64 375.92 0)
 			(hide yes)
@@
 			)
 		)
-		(property "Package" "0603"
+		(property "Package" "1206"
+			(at 40.64 375.92 0)
+			(hide yes)
+			(effects
+				(font (size 1.27 1.27))
+			)
+		)
+		(property "TCR" "25 ppm/K"
 			(at 40.64 375.92 0)
 			(hide yes)
@@
 			)
 		)
-		(property "Footprint" "Resistor_SMD:R_0603_1608Metric"
+		(property "Footprint" "Resistor_SMD:R_1206_3216Metric"
 			(at 50.8 375.92 0)
 			(hide yes)
@@
 			)
 		)
-		(property "Datasheet" "https://www.vishay.com/docs/20035/dcrcwe3.pdf"
+		(property "Datasheet" "https://www.vishay.com/docs/28758/tnpw_e3.pdf"
 			(at 50.8 375.92 0)
 			(hide yes)
@@
 			)
 		)
-		(property "Description" "Resistor 36.5k 1% 0603"
+		(property "Description" "Resistor 36.5k 0.1% 1206"
 			(at 50.8 375.92 0)
 			(hide yes)
@@
 			)
 		)
-		(property "MPN" "CRCW060336K5FKEA"
+		(property "MPN" "TNPW120636K5BEEA"
 			(at 50.8 375.92 0)
 			(hide yes)
@@
 			)
 		)
-		(property "Manufacturer" "Vishay Dale"
+		(property "Manufacturer" "Vishay Draloric"
 			(at 50.8 375.92 0)
 			(hide yes)
@@
 			)
 		)
-		(property "Tolerance" "1%"
+		(property "Tolerance" "0.1%"
 			(at 50.8 375.92 0)
 			(hide yes)
@@
 			)
 		)
-		(property "Package" "0603"
+		(property "Package" "1206"
+			(at 50.8 375.92 0)
+			(hide yes)
+			(effects
+				(font (size 1.27 1.27))
+			)
+		)
+		(property "TCR" "25 ppm/K"
 			(at 50.8 375.92 0)
 			(hide yes)
