File: designs/leadacid-balancer/out/ch3.kicad_sch (KiCad schematic)
At the start: 127 parts, among them Q301 CSD18543Q3A, Q302 CSD18543Q3A, Q303 CSD18543Q3A, Q304 CSD18543Q3A, Q305 MMBT3906, Q306 2N7002, Q307 MMBT3906, U301 UCC21520ADWR, U302 UCC21520ADWR, U303 CD4047BM96, U304 TPS7A1601DGNR, U305 TPS7A1601DGNR, U306 TPS70950DBVR, U307 REF35250, U308 TLV7044PWR, U309 74LVC1G02, U310 SFH617A-3

Commit message: designs: work-in-progress (review fixes under way)
Co-Authored-By: Claude Opus 5.5 <noreply@anthropic.com>
Claude-Session: https://claude.ai/code/session_01VFJn9VbX8h27kf4LpLwEtn
Parts:
- added C351: 4.7u, Capacitor_SMD:C_0805_2012Metric, symbol Device:C
- added C352: 100n, Capacitor_SMD:C_0603_1608Metric, symbol Device:C
- added C353, C354: 470n, Capacitor_SMD:C_0603_1608Metric, symbol Device:C
- added D305: BAS16W, Package_TO_SOT_SMD:SOT-323_SC-70, symbol Diode:BAS16W
- added JP302: EN, Connector_PinHeader_2.54mm:PinHeader_1x02_P2.54mm_Vertical, symbol Jumper:Jumper_2_Open
- added JS302: 60900213421, symbol Mechanical:Housing
- added R354, R355, R356, R357, R360, R361, R362, R363, R366, R367, R368, R369: 2M, Resistor_SMD:R_1206_3216Metric, symbol Device:R
- added R358, R359: 4.7, Resistor_SMD:R_0603_1608Metric, symbol Device:R
- added R364, R365: 1.62M, Resistor_SMD:R_1206_3216Metric, symbol Device:R
- added R370, R371: 1.7M, Resistor_SMD:R_1206_3216Metric, symbol Device:R
- added R372: 825, Resistor_SMD:R_0603_1608Metric, symbol Device:R
- added R373, R374, R375, R378, R379: 4.99M, Resistor_SMD:R_0603_1608Metric, symbol Device:R
- added R376: 100k, Resistor_SMD:R_0603_1608Metric, symbol Device:R
- added R377: 249k, Resistor_SMD:R_0603_1608Metric, symbol Device:R
- added unit 2 of U309
- added unit 3 of U309
- added U311: TLV7044PWR, Package_SO:TSSOP-14_4.4x5mm_P0.65mm, symbol kaesynth:TLV7044PWR
- C338: value 2.2u -> 4.7u; footprint Capacitor_SMD:C_0603_1608Metric -> Capacitor_SMD:C_0805_2012Metric; MPN GRM188R71C225KE11D -> GRM21BR71E475KA73L; Voltage 16V -> 25V
- R326, R327, R330, R331: value 4.99M -> 2M; footprint Resistor_SMD:R_0603_1608Metric -> Resistor_SMD:R_1206_3216Metric; MPN CRCW06034M99FKEA -> TNPW12062M00BEEA; Manufacturer Vishay Dale -> Vishay Draloric; Package 0603 -> 1206; TCR (none) -> 25 ppm/K; Tolerance 1% -> 0.1%
- R328, R329: value 1M -> 1.58M; footprint Resistor_SMD:R_0603_1608Metric -> Resistor_SMD:R_1206_3216Metric; MPN CRCW06031M00FKEA -> TNPW12061M58BEEA; Manufacturer Vishay Dale -> Vishay Draloric; Package 0603 -> 1206; TCR (none) -> 25 ppm/K; Tolerance 1% -> 0.1%
- R332, R333: value 1.1M -> 1.74M; footprint Resistor_SMD:R_0603_1608Metric -> Resistor_SMD:R_1206_3216Metric; MPN CRCW06031M10FKEA -> TNPW12061M74BEEA; Manufacturer Vishay Dale -> Vishay Draloric; Package 0603 -> 1206; TCR (none) -> 25 ppm/K; Tolerance 1% -> 0.1%
- R334, R335: value 2.26M -> 2M; footprint Resistor_SMD:R_0603_1608Metric -> Resistor_SMD:R_1206_3216Metric; MPN CRCW06032M26FKEA -> TNPW12062M00BEEA; Manufacturer Vishay Dale -> Vishay Draloric; Package 0603 -> 1206; TCR (none) -> 25 ppm/K; Tolerance 1% -> 0.1%
- R336, R337: value 1M -> 1.85M; footprint Resistor_SMD:R_0603_1608Metric -> Resistor_SMD:R_1206_3216Metric; MPN CRCW06031M00FKEA -> TNPW12061M85BEEA; Manufacturer Vishay Dale -> Vishay Draloric; Package 0603 -> 1206; TCR (none) -> 25 ppm/K; Tolerance 1% -> 0.1%
- R342: value 100k -> 10k; MPN CRCW0603100KFKEA -> CRCW060310K0FKEA
- R345: value 249 -> 750; MPN CRCW0603249RFKEA -> CRCW0603750RFKEA
- U309: value 74LVC1G02 -> 74LVC2G02; footprint Package_TO_SOT_SMD:SOT-23-5 -> Package_SO:SSOP-8_2.95x2.8mm_P0.65mm; symbol 74xGxx:74LVC1G02 -> 74xGxx:74LVC2G02; MPN SN74LVC1G02DBVR -> SN74LVC2G02DCTR
Connections:
- net ALM_E: now also JP302.2 (B)
- net CH3_12VL: now also R359.1; no longer D302.1 (A)
- net CH3_12VU: now also R358.1; no longer D301.1 (A)
- net CH3_FLT: now also U309.7, U309.6; no longer Q305.3 (C), R344.1, R345.1, U309.2
- net CH3_FLT_N: now also U309.1, U309.2
- net CH3_N: now also U311.5 (INB+), U311.9 (INC-)
- net CH3_NCHG: now also U309.5; no longer U309.1
- net CH3_PHI: now also R357.2; no longer R331.2
- net CH3_PLO: now also R355.2; no longer R327.2
- net CH3_RUN: now also R372.1, R376.1, U309.3; no longer U309.4
- net CH3_V5: now also C352.1, R373.1, U309.8 (VCC), U311.4 (VCC); no longer U309.5 (VCC)
- net CH3_VREF: now also U311.2 (INA-)
- net TAP2: now also D303.1 (K), C351.2, C352.2, C353.2, C354.2, R364.2, R365.2, R370.2, R371.2, R374.2, U309.4 (GND), U311.11 (VEE), U311.3 (INA+); no longer U301.5 (DIS), U302.5 (DIS), U309.3 (GND)
- net TAP4: now also R360.1, R366.1
- net ALM_C renamed ALM_S3
- net ALM_S3: now also JP302.1 (A)
- net CH3_N_M renamed CH3_N_M1
- net CH3_OPTO_A renamed CH3_OKA
- net CH3_OKA: now also R372.2, U311.7 (OUTB), U311.8 (OUTC); no longer D303.1 (K)
- net CH3_PHI_M renamed CH3_PHI_M1
- net CH3_PLO_M renamed CH3_PLO_M1
- net CH3_PON_A renamed CH3_PON_M1
- net CH3_PON_B renamed CH3_PON_M2
- net CH3_PON_C renamed CH3_PON_M3
- new net CH3_BSL_A: D302.1 (A), R359.2
- new net CH3_BSU_A: D301.1 (A), R358.2
- new net CH3_LEDQ: Q305.3 (C), R344.1, R345.1
- new net CH3_PAUSE: D305.1 (A), R375.1, R376.2, R378.1, U301.5 (DIS), U302.5 (DIS), U311.14 (OUTD)
- new net CH3_PDA: D305.3 (K), R377.1
- new net CH3_PHI_M2: R331.2, R356.1
- new net CH3_PHI_M3: R356.2, R357.1
- new net CH3_PLO_M2: R327.2, R354.1
- new net CH3_PLO_M3: R354.2, R355.1
- new net CH3_PWH: C353.1, R363.2, R364.1, R365.1, U311.6 (INB-)
- new net CH3_PWH_M1: R360.2, R361.1
- new net CH3_PWH_M2: R361.2, R362.1
- new net CH3_PWH_M3: R362.2, R363.1
- new net CH3_PWL: C354.1, R369.2, R370.1, R371.1, U311.10 (INC+)
- new net CH3_PWL_M1: R366.2, R367.1
- new net CH3_PWL_M2: R367.2, R368.1
- new net CH3_PWL_M3: R368.2, R369.1
- new net CH3_TCT: C351.1, R377.2, R379.2, U311.13 (IND-)
- new net CH3_TPN: R373.2, R374.1, R375.2, U311.12 (IND+)
- new net CH3_TSM: R378.2, R379.1
- no-connect marks 17 -> 19
Other:
- moved on the sheet: C301, C302, C303, C304, C305, C306, C307, C308, C309, C310, C311, C312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

Commit message: designs: work-in-progress (review fixes under way)
Co-Authored-By: Claude Opus 5.5 <noreply@anthropic.com>
Claude-Session: https://claude.ai/code/session_01VFJn9VbX8h27kf4LpLwEtn
Parts:
- removed R364, R365: 1.62M, Resistor_SMD:R_1206_3216Metric, symbol Device:R
- removed R366, R367, R368, R369: 2M, Resistor_SMD:R_1206_3216Metric, symbol Device:R
- removed R370, R371: 1.7M, Resistor_SMD:R_1206_3216Metric, symbol Device:R
- R332, R333: value 1.74M -> 1.7M; MPN TNPW12061M74BEEA -> TNPW12061M70BEEA
- R355: value 2M -> 1.96M; MPN TNPW12062M00BEEA -> TNPW12061M96BEEA
- R360, R361: value 2M -> 30.9k; footprint Resistor_SMD:R_1206_3216Metric -> Resistor_SMD:R_0603_1608Metric; MPN TNPW12062M00BEEA -> CRCW060330K9FKEA; Manufacturer Vishay Draloric -> Vishay Dale; Package 1206 -> 0603; TCR 25 ppm/K -> (none); Tolerance 0.1% -> 1%
- R362, R363: value 2M -> 36.5k; footprint Resistor_SMD:R_1206_3216Metric -> Resistor_SMD:R_0603_1608Metric; MPN TNPW12062M00BEEA -> CRCW060336K5FKEA; Manufacturer Vishay Draloric -> Vishay Dale; Package 1206 -> 0603; TCR 25 ppm/K -> (none); Tolerance 0.1% -> 1%
Connections:
- net CH3_PHI: now also R362.1, R363.1; no longer R332.1, R333.1
- net CH3_PLO: now also R360.2, R361.2; no longer R355.2
- net CH3_PWH: now also R355.2, R360.1, R361.1; no longer R363.2
- net CH3_PWL: now also R332.1, R333.1, R362.2, R363.2
- net TAP4: no longer R360.1
- removed net CH3_PWH_M1: R360.2, R361.1
- removed net CH3_PWH_M2: R361.2, R362.1
- removed net CH3_PWH_M3: R362.2, R363.1
Other:
- moved on the sheet: C301, C302, C303, C304, C305, C306, C307, C308, C309, C318, C326, C327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

Commit message: designs/leadacid-balancer: fix the independent review's blocker and majors
- B-1: board fuse KLKD006.T (6 A, 600 VDC, 10 kA DC, 63 A2s) in Keystone 3576 holders
  (custom footprint; board 180 x 130 mm); worst board fault 670 A vs 10 kA.
- M-1: 0.1 % thin-film supervisor strings; tolerance incl. comparator offset, half
  hysteresis and TCR is +/-1.34 % vs the 1.5 % budget; worst-case trip points in calcs.
- M-2: RUN = NOR(NCHG, FLT) on a logic gate; the fault transistor only drives the LED.
- M-3: +/-4 % imbalance warning opens the alarm; silent current into a failing battery
  <= 2.44 A (was 4.4 A).
- M-4: fail-safe alarm loop (closed only while all channels are healthy); periodic tap
  check catches a floating tap in 1.14 s.
- Minors fixed or answered. Build: 0 errors, ERC clean, netlist identical, 31 waived;
  N = 2/3 variants clean.

Co-Authored-By: Claude Opus 5.5 <noreply@anthropic.com>
Claude-Session: https://claude.ai/code/session_01VFJn9VbX8h27kf4LpLwEtn
Parts:
- R358, R359: value 4.7 -> 10; MPN CRCW06034R70FKEA -> CRCW060310R0FKEA
- R360, R361: footprint Resistor_SMD:R_0603_1608Metric -> Resistor_SMD:R_1206_3216Metric; MPN CRCW060330K9FKEA -> TNPW120630K9BEEA; Manufacturer Vishay Dale -> Vishay Draloric; Package 0603 -> 1206; TCR (none) -> 25 ppm/K; Tolerance 1% -> 0.1%
- R362, R363: footprint Resistor_SMD:R_0603_1608Metric -> Resistor_SMD:R_1206_3216Metric; MPN CRCW060336K5FKEA -> TNPW120636K5BEEA; Manufacturer Vishay Dale -> Vishay Draloric; Package 0603 -> 1206; TCR (none) -> 25 ppm/K; Tolerance 1% -> 0.1%
Changed lines of the file:
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@@
 			)
 		)
-		(property "Value" "4.7"
+		(property "Value" "10"
 			(at 370.84 180.34 90)
 			(effects
@@
 			)
 		)
-		(property "Description" "Resistor 4.7 1% 0603"
+		(property "Description" "Resistor 10 1% 0603"
 			(at 370.84 180.34 0)
 			(hide yes)
@@
 			)
 		)
-		(property "MPN" "CRCW06034R70FKEA"
+		(property "MPN" "CRCW060310R0FKEA"
 			(at 370.84 180.34 0)
 			(hide yes)
@@
 			)
 		)
-		(property "Value" "4.7"
+		(property "Value" "10"
 			(at 381 180.34 90)
 			(effects
@@
 			)
 		)
-		(property "Description" "Resistor 4.7 1% 0603"
+		(property "Description" "Resistor 10 1% 0603"
 			(at 381 180.34 0)
 			(hide yes)
@@
 			)
 		)
-		(property "MPN" "CRCW06034R70FKEA"
+		(property "MPN" "CRCW060310R0FKEA"
 			(at 381 180.34 0)
 			(hide yes)
@@
 			)
 		)
-		(property "Footprint" "Resistor_SMD:R_0603_1608Metric"
+		(property "Footprint" "Resistor_SMD:R_1206_3216Metric"
 			(at 73.66 322.58 0)
 			(hide yes)
@@
 			)
 		)
-		(property "Datasheet" "https://www.vishay.com/docs/20035/dcrcwe3.pdf"
+		(property "Datasheet" "https://www.vishay.com/docs/28758/tnpw_e3.pdf"
 			(at 73.66 322.58 0)
 			(hide yes)
@@
 			)
 		)
-		(property "Description" "Resistor 30.9k 1% 0603"
+		(property "Description" "Resistor 30.9k 0.1% 1206"
 			(at 73.66 322.58 0)
 			(hide yes)
@@
 			)
 		)
-		(property "MPN" "CRCW060330K9FKEA"
+		(property "MPN" "TNPW120630K9BEEA"
 			(at 73.66 322.58 0)
 			(hide yes)
@@
 			)
 		)
-		(property "Manufacturer" "Vishay Dale"
+		(property "Manufacturer" "Vishay Draloric"
 			(at 73.66 322.58 0)
 			(hide yes)
@@
 			)
 		)
-		(property "Tolerance" "1%"
+		(property "Tolerance" "0.1%"
 			(at 73.66 322.58 0)
 			(hide yes)
@@
 			)
 		)
-		(property "Package" "0603"
+		(property "Package" "1206"
+			(at 73.66 322.58 0)
+			(hide yes)
+			(effects
+				(font (size 1.27 1.27))
+			)
+		)
+		(property "TCR" "25 ppm/K"
 			(at 73.66 322.58 0)
 			(hide yes)
@@
 			)
 		)
-		(property "Footprint" "Resistor_SMD:R_0603_1608Metric"
+		(property "Footprint" "Resistor_SMD:R_1206_3216Metric"
 			(at 86.36 322.58 0)
 			(hide yes)
@@
 			)
 		)
-		(property "Datasheet" "https://www.vishay.com/docs/20035/dcrcwe3.pdf"
+		(property "Datasheet" "https://www.vishay.com/docs/28758/tnpw_e3.pdf"
 			(at 86.36 322.58 0)
 			(hide yes)
@@
 			)
 		)
-		(property "Description" "Resistor 30.9k 1% 0603"
+		(property "Description" "Resistor 30.9k 0.1% 1206"
 			(at 86.36 322.58 0)
 			(hide yes)
@@
 			)
 		)
-		(property "MPN" "CRCW060330K9FKEA"
+		(property "MPN" "TNPW120630K9BEEA"
 			(at 86.36 322.58 0)
 			(hide yes)
@@
 			)
 		)
-		(property "Manufacturer" "Vishay Dale"
+		(property "Manufacturer" "Vishay Draloric"
 			(at 86.36 322.58 0)
 			(hide yes)
@@
 			)
 		)
-		(property "Tolerance" "1%"
+		(property "Tolerance" "0.1%"
 			(at 86.36 322.58 0)
 			(hide yes)
@@
 			)
 		)
-		(property "Package" "0603"
+		(property "Package" "1206"
+			(at 86.36 322.58 0)
+			(hide yes)
+			(effects
+				(font (size 1.27 1.27))
+			)
+		)
+		(property "TCR" "25 ppm/K"
 			(at 86.36 322.58 0)
 			(hide yes)
@@
 			)
 		)
-		(property "Footprint" "Resistor_SMD:R_0603_1608Metric"
+		(property "Footprint" "Resistor_SMD:R_1206_3216Metric"
 			(at 40.64 375.92 0)
 			(hide yes)
@@
 			)
 		)
-		(property "Datasheet" "https://www.vishay.com/docs/20035/dcrcwe3.pdf"
+		(property "Datasheet" "https://www.vishay.com/docs/28758/tnpw_e3.pdf"
 			(at 40.64 375.92 0)
 			(hide yes)
@@
 			)
 		)
-		(property "Description" "Resistor 36.5k 1% 0603"
+		(property "Description" "Resistor 36.5k 0.1% 1206"
 			(at 40.64 375.92 0)
 			(hide yes)
@@
 			)
 		)
-		(property "MPN" "CRCW060336K5FKEA"
+		(property "MPN" "TNPW120636K5BEEA"
 			(at 40.64 375.92 0)
 			(hide yes)
@@
 			)
 		)
-		(property "Manufacturer" "Vishay Dale"
+		(property "Manufacturer" "Vishay Draloric"
 			(at 40.64 375.92 0)
 			(hide yes)
@@
 			)
 		)
-		(property "Tolerance" "1%"
+		(property "Tolerance" "0.1%"
 			(at 40.64 375.92 0)
 			(hide yes)
@@
 			)
 		)
-		(property "Package" "0603"
+		(property "Package" "1206"
+			(at 40.64 375.92 0)
+			(hide yes)
+			(effects
+				(font (size 1.27 1.27))
+			)
+		)
+		(property "TCR" "25 ppm/K"
 			(at 40.64 375.92 0)
 			(hide yes)
@@
 			)
 		)
-		(property "Footprint" "Resistor_SMD:R_0603_1608Metric"
+		(property "Footprint" "Resistor_SMD:R_1206_3216Metric"
 			(at 50.8 375.92 0)
 			(hide yes)
@@
 			)
 		)
-		(property "Datasheet" "https://www.vishay.com/docs/20035/dcrcwe3.pdf"
+		(property "Datasheet" "https://www.vishay.com/docs/28758/tnpw_e3.pdf"
 			(at 50.8 375.92 0)
 			(hide yes)
@@
 			)
 		)
-		(property "Description" "Resistor 36.5k 1% 0603"
+		(property "Description" "Resistor 36.5k 0.1% 1206"
 			(at 50.8 375.92 0)
 			(hide yes)
@@
 			)
 		)
-		(property "MPN" "CRCW060336K5FKEA"
+		(property "MPN" "TNPW120636K5BEEA"
 			(at 50.8 375.92 0)
 			(hide yes)
@@
 			)
 		)
-		(property "Manufacturer" "Vishay Dale"
+		(property "Manufacturer" "Vishay Draloric"
 			(at 50.8 375.92 0)
 			(hide yes)
@@
 			)
 		)
-		(property "Tolerance" "1%"
+		(property "Tolerance" "0.1%"
 			(at 50.8 375.92 0)
 			(hide yes)
@@
 			)
 		)
-		(property "Package" "0603"
+		(property "Package" "1206"
+			(at 50.8 375.92 0)
+			(hide yes)
+			(effects
+				(font (size 1.27 1.27))
+			)
+		)
+		(property "TCR" "25 ppm/K"
 			(at 50.8 375.92 0)
 			(hide yes)
