File: designs/liion-balancer/out/afe.kicad_sch (KiCad schematic)
At the start: 19 parts, among them U1 ADBMS1818ASWZ

Commit message: designs: work-in-progress (review fixes under way)
Co-Authored-By: Claude Opus 5.5 <noreply@anthropic.com>
Claude-Session: https://claude.ai/code/session_01VFJn9VbX8h27kf4LpLwEtn
Parts:
- added C22: 100n, Capacitor_SMD:C_0603_1608Metric, symbol Device:C
- added R29: 10.0k, Resistor_SMD:R_0603_1608Metric, symbol Device:R
- added TH4: 10k, Resistor_SMD:R_0603_1608Metric, symbol Device:Thermistor_NTC
Connections:
- net GND_B: now also C22.2, TH4.2; no longer U1.42 (GPIO4)
- net VREF2: now also R29.1
- new net NTC4: C22.1, R29.2, TH4.1, U1.42 (GPIO4)
Other:
- moved on the sheet: C5, C6, C7, TH1, TH2, TH3, U1B
