File: designs/liion-balancer/out/ch12.kicad_sch (KiCad schematic)
At the start: 15 parts, among them T112 NA5743-ALD, U112 LT8584EFE#PBF, U212 TLP293(GB)

Commit message: designs: work-in-progress (review fixes under way)
Co-Authored-By: Claude Opus 5.5 <noreply@anthropic.com>
Claude-Session: https://claude.ai/code/session_01VFJn9VbX8h27kf4LpLwEtn
Parts:
- added R512: 10k, Resistor_SMD:R_0603_1608Metric, symbol Device:R
Connections:
- net S_12: now also R512.1; no longer U112.7 (DIN)
- new net DIN_12: R512.2, U112.7 (DIN)
Other:
- moved on the sheet: C612, D112, T112, U212
