File: designs/liion-balancer/out/ch13.kicad_sch (KiCad schematic)
At the start: 15 parts, among them T113 NA5743-ALD, U113 LT8584EFE#PBF, U213 TLP293(GB)

Commit message: designs: work-in-progress (review fixes under way)
Co-Authored-By: Claude Opus 5.5 <noreply@anthropic.com>
Claude-Session: https://claude.ai/code/session_01VFJn9VbX8h27kf4LpLwEtn
Parts:
- added R513: 10k, Resistor_SMD:R_0603_1608Metric, symbol Device:R
Connections:
- net S_13: now also R513.1; no longer U113.7 (DIN)
- new net DIN_13: R513.2, U113.7 (DIN)
Other:
- moved on the sheet: C613, D113, T113, U213
