File: designs/liion-balancer/out/ch14.kicad_sch (KiCad schematic)
At the start: 15 parts, among them T114 NA5743-ALD, U114 LT8584EFE#PBF, U214 TLP293(GB)

Commit message: designs: work-in-progress (review fixes under way)
Co-Authored-By: Claude Opus 5.5 <noreply@anthropic.com>
Claude-Session: https://claude.ai/code/session_01VFJn9VbX8h27kf4LpLwEtn
Parts:
- added R514: 10k, Resistor_SMD:R_0603_1608Metric, symbol Device:R
Connections:
- net S_14: now also R514.1; no longer U114.7 (DIN)
- new net DIN_14: R514.2, U114.7 (DIN)
Other:
- moved on the sheet: C614, D114, T114, U214
