File: designs/liion-balancer/out/ch15.kicad_sch (KiCad schematic)
At the start: 15 parts, among them T115 NA5743-ALD, U115 LT8584EFE#PBF, U215 TLP293(GB)

Commit message: designs: work-in-progress (review fixes under way)
Co-Authored-By: Claude Opus 5.5 <noreply@anthropic.com>
Claude-Session: https://claude.ai/code/session_01VFJn9VbX8h27kf4LpLwEtn
Parts:
- added R515: 10k, Resistor_SMD:R_0603_1608Metric, symbol Device:R
Connections:
- net S_15: now also R515.1; no longer U115.7 (DIN)
- new net DIN_15: R515.2, U115.7 (DIN)
Other:
- moved on the sheet: C615, D115, T115, U215
