File: designs/liion-balancer/out/ch16.kicad_sch (KiCad schematic)
At the start: 15 parts, among them T116 NA5743-ALD, U116 LT8584EFE#PBF, U216 TLP293(GB)

Commit message: designs: work-in-progress (review fixes under way)
Co-Authored-By: Claude Opus 5.5 <noreply@anthropic.com>
Claude-Session: https://claude.ai/code/session_01VFJn9VbX8h27kf4LpLwEtn
Parts:
- added R516: 10k, Resistor_SMD:R_0603_1608Metric, symbol Device:R
Connections:
- net S_16: now also R516.1; no longer U116.7 (DIN)
- new net DIN_16: R516.2, U116.7 (DIN)
Other:
- moved on the sheet: C616, D116, T116, U216
