File: designs/liion-balancer/out/en.kicad_sch (KiCad schematic)
At the start: 7 parts, among them Q1 MMBT5551

Commit message: designs: work-in-progress (review fixes under way)
Co-Authored-By: Claude Opus 5.5 <noreply@anthropic.com>
Claude-Session: https://claude.ai/code/session_01VFJn9VbX8h27kf4LpLwEtn
Parts:
- added D10, D9: BZX84-B3V9, Package_TO_SOT_SMD:SOT-23, symbol Diode:BZX84Cxx
- added D8: ES1G-13-F, Diode_SMD:D_SMA, symbol Device:D
- added Q2: MMBT5551, Package_TO_SOT_SMD:SOT-23, symbol Transistor_BJT:MMBT5551L
- added R30, R31: 220, Resistor_SMD:R_0603_1608Metric, symbol Device:R
- added R32, R36, R37: 10k, Resistor_SMD:R_0603_1608Metric, symbol Device:R
- added R33: 100k, Resistor_SMD:R_0603_1608Metric, symbol Device:R
- added U10, U9: TLP293(GB), Package_SO:SOIC-4_4.55x2.6mm_P1.27mm, symbol Isolator:TLP293
Connections:
- net BAL_EN: now also R32.1
- net GND_B: now also Q2.2 (E), R33.2, U10.3, U9.3
- net Q1_B: now also U10.4, U9.4; no longer R21.2
- new net EN_MCU: R21.2
- new net FLYBUS: D8.2 (A)
- new net Q2_B: Q2.1 (B), R32.2, R33.1
- new net TAP1: D10.3 (K)
- new net TAP15: R36.2, U9.2
- new net TRB1: D10.1 (A), R31.1
- new net TRB2: R31.2, R37.1, U10.1
- new net TRB3: Q2.3 (C), R37.2, U10.2
- new net TRT1: D8.1 (K), D9.3 (K)
- new net TRT2: D9.1 (A), R30.1
- new net TRT3: R30.2, R36.1, U9.1
- no-connect marks 0 -> 2
Other:
- title: Global balance enable: Q1 current sink and the 16-LED opto string -> Balance enable: Q1 sink, opto string, hardware trips
- moved on the sheet: D4, R21, R22, R23, R24, TP5
