File: designs/liion-balancer/out/iso.kicad_sch (KiCad schematic)
At the start: 12 parts, among them J2 1803293, J4 1803277, U5 ISO7721DWV, U6 AQY210EHAX, U7 TPD4E05U06

Commit message: designs: work-in-progress (review fixes under way)
Co-Authored-By: Claude Opus 5.5 <noreply@anthropic.com>
Claude-Session: https://claude.ai/code/session_01VFJn9VbX8h27kf4LpLwEtn
Parts:
- added D11: ES1G-13-F, Diode_SMD:D_SMA, symbol Device:D
- added D12: SMBJ40CA, Diode_SMD:D_SMB, symbol Device:D_TVS
- added J5: 1803277, Connector_Phoenix_MC:PhoenixContact_MC_1,5_2-G-3.81_1x02_P3.81mm_Horizontal, symbol Connector_Generic:Conn_01x02
- added R34: 1.8k, Resistor_SMD:R_2512_6332Metric, symbol Device:R
- added R35: 10k, Resistor_SMD:R_0603_1608Metric, symbol Device:R
- added U8: AQY210EHAX, Package_DIP:SMDIP-4_W7.62mm, symbol Relay_SolidState:AQY280EH
Connections:
- new net BMS1: D11.2 (A), R34.2
- new net BMS2: D11.1 (K), R35.1, U8.1
- new net BMS_IN: D12.1 (A1), J5.1 (Pin_1), R34.1
- new net BMS_N: D12.2 (A2), J5.2 (Pin_2), R35.2, U8.2
- new net EN_MCU: U8.3
- new net Q1_B: U8.4
Other:
- moved on the sheet: J2
