File: designs/liion-balancer/out/psu.kicad_sch (KiCad schematic)
At the start: 22 parts, among them U3 LM5164, U4 MCP1700-3.3

Commit message: designs: work-in-progress (review fixes under way)
Co-Authored-By: Claude Opus 5.5 <noreply@anthropic.com>
Claude-Session: https://claude.ai/code/session_01VFJn9VbX8h27kf4LpLwEtn
Parts:
- R10: value 4.7M -> 10M; MPN RC1206FR-074M7L -> RC1206FR-0710ML
- R11: value 300k -> 620k; MPN RC0603FR-07300KL -> RC0603FR-07620KL
Changed lines of the file:
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@@
 			)
 		)
-		(property "Value" "4.7M"
+		(property "Value" "10M"
 			(at 66.04 93.98 90)
 			(effects
@@
 			)
 		)
-		(property "Description" "Resistor 4.7M 1% 1206"
+		(property "Description" "Resistor 10M 1% 1206"
 			(at 66.04 93.98 0)
 			(hide yes)
@@
 			)
 		)
-		(property "MPN" "RC1206FR-074M7L"
+		(property "MPN" "RC1206FR-0710ML"
 			(at 66.04 93.98 0)
 			(hide yes)
@@
 			)
 		)
-		(property "Value" "300k"
+		(property "Value" "620k"
 			(at 76.2 93.98 90)
 			(effects
@@
 			)
 		)
-		(property "Description" "Resistor 300k 1% 0603"
+		(property "Description" "Resistor 620k 1% 0603"
 			(at 76.2 93.98 0)
 			(hide yes)
@@
 			)
 		)
-		(property "MPN" "RC0603FR-07300KL"
+		(property "MPN" "RC0603FR-07620KL"
 			(at 76.2 93.98 0)
 			(hide yes)
