File: designs/liion-balancer/out/ret.kicad_sch (KiCad schematic)
At the start: 6 parts

Commit message: designs: work-in-progress (review fixes under way)
Co-Authored-By: Claude Opus 5.5 <noreply@anthropic.com>
Claude-Session: https://claude.ai/code/session_01VFJn9VbX8h27kf4LpLwEtn
Parts:
- removed D2: SMBJ70A, Diode_SMD:D_SMB, symbol Device:D_Zener
- R19: value 2.0M -> 10M; MPN RC1206FR-072ML -> RC1206FR-0710ML
- R20: value 100k -> 470k; MPN RC0603FR-07100KL -> RC0603FR-07470KL
Other:
- title: Stack return: D1 blocking diode, D2 clamp, FLYBUS sense -> Stack return: D1 blocking diode and FLYBUS sense
- moved on the sheet: C19, R19, R20, TP1
