File: designs/prius-solar-mppt/out/DCX.kicad_sch (KiCad schematic)
At the start: 80 parts, among them J301 1766356, Q301 IAUC100N10, Q302 IAUC100N10, T301 T301-ETD39-DCX22 (custom), U301 UCC27282QDRCRQ1

Commit message: designs/prius-solar-mppt: v0.3, fix the independent review's blockers and majors
- B1: CHASSIS domain with reinforced DC barriers to HV and PACK (10/8 mm), HV/PACK edge
  clearance 10 mm, mounting holes fixed with 13 mm keep-outs; thermal pedestal under LV
  parts only.
- B2: no primary source for the Prime's full-charge cell voltage was found (blocking
  Q-13); hardware clamp set below a 4.00 V/cell floor (L3 3.927 V, worst 3.963 V; L2
  3.836 V; L1 3.79 V) with DNP trim to raise later; until then charging may stop near
  55-65 % SOC.
- Majors: sink clamp + burst disable + PV-node trip and TVS against LM5176 reverse power;
  20 MHz AEC-Q200 crystal for CAN (listen-only start); parked insulation monitoring via a
  110 M bridge (also detects a welded relay); open-sensor-safe hardware OT; CAGE CLAMP HV
  terminals with a lid-switch HVIL; DCX on-time and 17.6 A primary overcurrent latches;
  supercap-held latch that clears overnight.
- Build: 0 errors, ERC clean, system and both board netlists identical; 9 waivers (17
  findings, was 32).

Co-Authored-By: Claude Opus 5.5 <noreply@anthropic.com>
Claude-Session: https://claude.ai/code/session_01VFJn9VbX8h27kf4LpLwEtn
Parts:
- added C361, C362, C363: 1n, Capacitor_SMD:C_0603_1608Metric, symbol Device:C
- added D305, D306: BAT46WJ, Diode_SMD:D_SOD-323F, symbol Diode:BAT46
- added L301: 0.56u, Inductor_SMD:L_Coilcraft_XAL7070-XXX, symbol Device:L
- added R311: 5m, Resistor_SMD:R_Shunt_Vishay_WSK2512_6332Metric_T1.19mm, symbol Device:R_Shunt
- added R312: 1k, Resistor_SMD:R_0603_1608Metric, symbol Device:R
- added R313, R314: 10k, Resistor_SMD:R_0603_1608Metric, symbol Device:R
- J301: value 1766356 -> 236-303; footprint Connector_Phoenix_GMSTB:PhoenixContact_GMSTBA_2,5_3-G-7,62_1x03_P7.62mm_Horizontal -> TerminalBlock_WAGO:TerminalBlock_WAGO_236-303_1x03_P10.00mm_45Degree; MPN 1766356 -> 236-303; Manufacturer Phoenix Contact -> WAGO
Connections:
- net GND: now also C361.2, C362.2, C363.2, R311.3, R311.4; no longer Q302.1 (S), Q302.2 (S), Q302.3 (S)
- net HB_SW: now also L301.1; no longer T301.1 (P_START), T301.2 (P_START)
- net HI_F: now also D305.1 (K), R313.1
- net LI_F: now also D306.1 (K), R314.1
- new net DCX_CS: C361.1, R312.2
- new net DCX_CSK: R311.2, R312.1
- new net DCX_RS: Q302.1 (S), Q302.2 (S), Q302.3 (S), R311.1
- new net HB_LR: L301.2, T301.1 (P_START), T301.2 (P_START)
- new net ONT_H: C362.1, D305.2 (A), R313.2
- new net ONT_L: C363.1, D306.2 (A), R314.2
Other:
- moved on the sheet: C311, C312, C313, C314, C315, C316, C317, C318, C319, C320, C321, C322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
