File: designs/prius-solar-mppt/out/board-main/HVSENSE.kicad_sch (KiCad schematic)
At the start: 76 parts, among them U401 AMC3330QDWERQ1, U402 TLV9001-Q1, U421 AMC3330QDWERQ1, U422 TLV9001-Q1, U441 AMC3302QDWERQ1, U442 TLV9001-Q1

Commit message: designs/prius-solar-mppt: v0.3, fix the independent review's blockers and majors
- B1: CHASSIS domain with reinforced DC barriers to HV and PACK (10/8 mm), HV/PACK edge
  clearance 10 mm, mounting holes fixed with 13 mm keep-outs; thermal pedestal under LV
  parts only.
- B2: no primary source for the Prime's full-charge cell voltage was found (blocking
  Q-13); hardware clamp set below a 4.00 V/cell floor (L3 3.927 V, worst 3.963 V; L2
  3.836 V; L1 3.79 V) with DNP trim to raise later; until then charging may stop near
  55-65 % SOC.
- Majors: sink clamp + burst disable + PV-node trip and TVS against LM5176 reverse power;
  20 MHz AEC-Q200 crystal for CAN (listen-only start); parked insulation monitoring via a
  110 M bridge (also detects a welded relay); open-sensor-safe hardware OT; CAGE CLAMP HV
  terminals with a lid-switch HVIL; DCX on-time and 17.6 A primary overcurrent latches;
  supercap-held latch that clears overnight.
- Build: 0 errors, ERC clean, system and both board netlists identical; 9 waivers (17
  findings, was 32).

Co-Authored-By: Claude Opus 5.5 <noreply@anthropic.com>
Claude-Session: https://claude.ai/code/session_01VFJn9VbX8h27kf4LpLwEtn
Parts:
- added C433: 10n, Capacitor_SMD:C_0603_1608Metric, symbol Device:C
- added R434: 10k, Resistor_SMD:R_0603_1608Metric, symbol Device:R
- R429, R431: value 12.1k -> 12.7k; MPN TNPW060312K1BEEA -> TNPW060312K7BEEA
Connections:
- net GND: now also C433.2
- net H2_DA_OUT: now also R434.1
- new net HV_V2_LIM: C433.1, R434.2
Other:
- moved on the sheet: C451, C452, C453, R401, R402, R421, R422, R423, R424, R425, R445, R447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
