File: designs/prius-solar-mppt/out/board-main/LIMIT.kicad_sch (KiCad schematic)
At the start: 22 parts, among them U801 2.500V 0.2%, U802 TLV9062-Q1

Commit message: designs/prius-solar-mppt: v0.3, fix the independent review's blockers and majors
- B1: CHASSIS domain with reinforced DC barriers to HV and PACK (10/8 mm), HV/PACK edge
  clearance 10 mm, mounting holes fixed with 13 mm keep-outs; thermal pedestal under LV
  parts only.
- B2: no primary source for the Prime's full-charge cell voltage was found (blocking
  Q-13); hardware clamp set below a 4.00 V/cell floor (L3 3.927 V, worst 3.963 V; L2
  3.836 V; L1 3.79 V) with DNP trim to raise later; until then charging may stop near
  55-65 % SOC.
- Majors: sink clamp + burst disable + PV-node trip and TVS against LM5176 reverse power;
  20 MHz AEC-Q200 crystal for CAN (listen-only start); parked insulation monitoring via a
  110 M bridge (also detects a welded relay); open-sensor-safe hardware OT; CAGE CLAMP HV
  terminals with a lid-switch HVIL; DCX on-time and 17.6 A primary overcurrent latches;
  supercap-held latch that clears overnight.
- Build: 0 errors, ERC clean, system and both board netlists identical; 9 waivers (17
  findings, was 32).

Co-Authored-By: Claude Opus 5.5 <noreply@anthropic.com>
Claude-Session: https://claude.ai/code/session_01VFJn9VbX8h27kf4LpLwEtn
Parts:
- added C808: 1u, Capacitor_SMD:C_0603_1608Metric, symbol Device:C
- added C809, C810: 100n, Capacitor_SMD:C_0603_1608Metric, symbol Device:C
- added C811: 10n, Capacitor_SMD:C_0603_1608Metric, symbol Device:C
- added D803: BAT46WJ, Diode_SMD:D_SOD-323F, symbol Diode:BAT46
- added R812: 866, Resistor_SMD:R_0603_1608Metric, symbol Device:R
- added R813, R815, R817: 10k, Resistor_SMD:R_0603_1608Metric, symbol Device:R
- added R814, R818: 100k, Resistor_SMD:R_0603_1608Metric, symbol Device:R
- added R816: 2.67k, Resistor_SMD:R_0603_1608Metric, symbol Device:R
- added U803: TLV9062-Q1, Package_SO:SOIC-8_3.9x4.9mm_P1.27mm, symbol Amplifier_Operational:TLV9062xD
- R802: value 1.5k -> 3.24k; MPN TNPW06031K50BEEA -> TNPW06033K24BEEA
Connections:
- net +3V3: now also C810.1, U803.8 (V+)
- net GND: now also C809.2, C810.2, C811.2, R813.2, R817.2, U803.4 (V-), U803.5 (+)
- net LIM: now also D803.1 (K)
- net VREF_CV: now also R818.2
- net VREF_LIM: now also R812.1, R816.1, R818.1
- new net CV2_N: C808.1, R814.2, U803.2 (-)
- new net CV2_OUT: D803.2 (A), R815.2, U803.1
- new net CV2_RZ: C808.2, R815.1
- new net HV_V2_LIM: U803.3 (+)
- new net U803B_FB: U803.6 (-), U803.7
- new net VREF_CV2: C809.1, R814.1, R816.2, R817.1
- new net VTH_BURST: C811.1, R812.2, R813.1
Other:
- title: L2 analog limiter: CV on pack voltage, CC on charge current (firmware-free) -> L2 analog limiter: CV on pack voltage (paths 1 and 2), CC on charge current (firmware-free)
- moved on the sheet: C802, C803, C807, R803, R804, R805, R810, R811, U802B, U802C
