File: designs/prius-solar-mppt/out/board-main/MCU.kicad_sch (KiCad schematic)
At the start: 52 parts, among them J701 61300611121, J702 1757242, J703 1757255, J704 43650-0215, J706 1757284, J707 1757255, Q701 MMBTA42, Q702 MMBTA42, Q703 MMBTA42, U701 DSPIC33CK256MP505-E/PT, U702 SN65HVD230Q-Q1, U703 25LC256

Commit message: designs/prius-solar-mppt: v0.3, fix the independent review's blockers and majors
- B1: CHASSIS domain with reinforced DC barriers to HV and PACK (10/8 mm), HV/PACK edge
  clearance 10 mm, mounting holes fixed with 13 mm keep-outs; thermal pedestal under LV
  parts only.
- B2: no primary source for the Prime's full-charge cell voltage was found (blocking
  Q-13); hardware clamp set below a 4.00 V/cell floor (L3 3.927 V, worst 3.963 V; L2
  3.836 V; L1 3.79 V) with DNP trim to raise later; until then charging may stop near
  55-65 % SOC.
- Majors: sink clamp + burst disable + PV-node trip and TVS against LM5176 reverse power;
  20 MHz AEC-Q200 crystal for CAN (listen-only start); parked insulation monitoring via a
  110 M bridge (also detects a welded relay); open-sensor-safe hardware OT; CAGE CLAMP HV
  terminals with a lid-switch HVIL; DCX on-time and 17.6 A primary overcurrent latches;
  supercap-held latch that clears overnight.
- Build: 0 errors, ERC clean, system and both board netlists identical; 9 waivers (17
  findings, was 32).

Co-Authored-By: Claude Opus 5.5 <noreply@anthropic.com>
Claude-Session: https://claude.ai/code/session_01VFJn9VbX8h27kf4LpLwEtn
Parts:
- added C719, C720: 10p, Capacitor_SMD:C_0603_1608Metric, symbol Device:C
- added J705: 1757242, Connector_Phoenix_MSTB:PhoenixContact_MSTBA_2,5_2-G-5,08_1x02_P5.08mm_Horizontal, symbol Connector_Generic:Conn_01x02
- added J708: 1757255, Connector_Phoenix_MSTB:PhoenixContact_MSTBA_2,5_3-G-5,08_1x03_P5.08mm_Horizontal, symbol Connector_Generic:Conn_01x03
- added NT701: NetTie, NetTie:NetTie-2_SMD_Pad0.5mm, symbol Device:NetTie_2
- added Y701: 20MHz, Crystal:Crystal_SMD_3225-4Pin_3.2x2.5mm, symbol Device:Crystal_GND24
- J706: value 1757284 -> 1757255; footprint Connector_Phoenix_MSTB:PhoenixContact_MSTBA_2,5_6-G-5,08_1x06_P5.08mm_Horizontal -> Connector_Phoenix_MSTB:PhoenixContact_MSTBA_2,5_3-G-5,08_1x03_P5.08mm_Horizontal; symbol Connector_Generic:Conn_01x06 -> Connector_Generic:Conn_01x03; MPN 1757284 -> 1757255
Connections:
- net LATCH_Q is gone; now on net NTC_HS: U701.26 (RB3/AN8)
- net AUX12: now also J705.1 (Pin_1); no longer J703.1 (Pin_1)
- net EE_CS_N: now also U701.37 (RB9/RP41); no longer U701.33 (RB5/PGD3)
- net GND: now also J706.3 (Pin_3), C719.2, C720.2, J708.3 (Pin_3), NT701.2, Y701.2 (G), Y701.4 (G); no longer H701.1, H702.1, H703.1, H704.1, J706.5 (Pin_5), J706.6 (Pin_6)
- net NTC_HS: no longer U701.21 (RB0/AN5)
- net NTC_P3: now also U701.35 (RB7/AN2), J708.1 (Pin_1); no longer J706.3 (Pin_3), U701.22 (RB1/AN6)
- net NTC_P4: now also J708.2 (Pin_2); no longer J706.4 (Pin_4)
- net PERMIT_SNS: now also U701.47 (RB12/RP44); no longer U701.35 (RB7/TDO)
- net PGC: now also U701.34 (RB6/PGC3); no longer U701.37 (RB9/PGC1)
- net PGD: now also U701.33 (RB5/PGD3); no longer U701.36 (RB8/PGD1)
- net WDI: now also U701.45 (RB10/RP42); no longer U701.34 (RB6/PGC3)
- net LATCH_SNS: now reaches U701.46 (RB11/RP43)
- net IMD_SW: now reaches U701.48 (RB13/RP45)
- net UART_TX: no longer names the net of J701.6 (Pin_6)
- net UART_TX: no longer U701.45 (RB10/TMS)
- new net CHASSIS: H701.1, H702.1, H703.1, H704.1, NT701.1
- new net HVIL_A: J703.1 (Pin_1), J705.2 (Pin_2)
- new net IMD_ADC: U701.36 (RB8/AN10)
- new net XTAL_I: C719.1, U701.21 (OSCI/RB0), Y701.1
- new net XTAL_O: C720.1, U701.22 (OSCO/RB1), Y701.3
- no-connect marks 5 -> 3
Other:
- moved on the sheet: C701, C702, C703, C704, C705, C706, C707, C714, C715, C716, C717, C718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
