File: designs/prius-solar-mppt/out/board-main/SAFETY.kicad_sch (KiCad schematic)
At the start: 49 parts, among them U501 2.500V 0.2%, U502 LM2901B-Q1, U503 SN74LVC2G74-Q1, U504 TPS3850G33QDRCRQ1, U505 TPL7407LA-Q1, U506 LM2901B-Q1

Commit message: designs/prius-solar-mppt: rework for the 2017 Prius Prime (Li-ion), charging car on and off
User decisions (2026-10-23): it is a Prius Prime with the Li-ion pack; it must charge
with the car on or off, be smart, and be weak enough that the pack cannot get into
trouble (stop by 80 %, voltage clamp, temperature compensation).

- Pack: 95 cells in series; no Prius pack is split while off (relays sit on the two pack
  cables; the service plug splits it only when pulled), so one tap pair on the cell side
  of the system main relays, fused on both poles, reaches the whole pack.
- Weak by construction: charge current capped at 0.30 A (>= 2 sun-days from 80 % to 100 %
  with firmware dead), analog CV/CC limiter on its own reference, latching overcurrent
  and overvoltage trips, 1:22 isolating DC transformer stage, 600 V relays, pack-sense
  core in the harness, event log, CAN transmit gated by ignition.
- Toyota's 180 W Prius PHV solar roof ("pump charging" through a buffer battery and the
  car's battery ECU) documented as the reference; this board does that ECU's job itself.
- Encoded in kaesynth: main (470 parts) and battery-end (15) boards, both netlists
  identical to the IR; 0 errors, 32 waived. The checks caught two v0.1 errors: an
  inverted UVLO (the stage never turned off) and the MPPT current sink on the wrong input.
- Blocking: roof measurement, junction-block tap location, installer/legality, roof
  fixing, and Q-10.

Co-Authored-By: Claude Opus 5.5 <noreply@anthropic.com>
Claude-Session: https://claude.ai/code/session_01VFJn9VbX8h27kf4LpLwEtn
Parts:
- R520: value 10k -> 100k; MPN ERJ-3EKF1002V -> ERJ-3EKF1003V
Changed lines of the file:
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@@
 			)
 		)
-		(property "Value" "10k"
+		(property "Value" "100k"
 			(at 27.94 287.02 90)
 			(effects
@@
 			)
 		)
-		(property "Description" "Resistor 10k 1% 0603"
+		(property "Description" "Resistor 100k 1% 0603"
 			(at 27.94 287.02 0)
 			(hide yes)
@@
 			)
 		)
-		(property "MPN" "ERJ-3EKF1002V"
+		(property "MPN" "ERJ-3EKF1003V"
 			(at 27.94 287.02 0)
 			(hide yes)

Commit message: designs/prius-solar-mppt: v0.3, fix the independent review's blockers and majors
- B1: CHASSIS domain with reinforced DC barriers to HV and PACK (10/8 mm), HV/PACK edge
  clearance 10 mm, mounting holes fixed with 13 mm keep-outs; thermal pedestal under LV
  parts only.
- B2: no primary source for the Prime's full-charge cell voltage was found (blocking
  Q-13); hardware clamp set below a 4.00 V/cell floor (L3 3.927 V, worst 3.963 V; L2
  3.836 V; L1 3.79 V) with DNP trim to raise later; until then charging may stop near
  55-65 % SOC.
- Majors: sink clamp + burst disable + PV-node trip and TVS against LM5176 reverse power;
  20 MHz AEC-Q200 crystal for CAN (listen-only start); parked insulation monitoring via a
  110 M bridge (also detects a welded relay); open-sensor-safe hardware OT; CAGE CLAMP HV
  terminals with a lid-switch HVIL; DCX on-time and 17.6 A primary overcurrent latches;
  supercap-held latch that clears overnight.
- Build: 0 errors, ERC clean, system and both board netlists identical; 9 waivers (17
  findings, was 32).

Co-Authored-By: Claude Opus 5.5 <noreply@anthropic.com>
Claude-Session: https://claude.ai/code/session_01VFJn9VbX8h27kf4LpLwEtn
Parts:
- removed C507: 100n, Capacitor_SMD:C_0603_1608Metric, symbol Device:C
- added C514, C518: 10n, Capacitor_SMD:C_0603_1608Metric, symbol Device:C
- added C515, C516, C517, C519, C522: 100n, Capacitor_SMD:C_0603_1608Metric, symbol Device:C
- added C521: 0.1F, Capacitor_THT:CP_Radial_D13.0mm_P5.00mm, symbol Device:C_Polarized
- added C523: 1u, Capacitor_SMD:C_0603_1608Metric, symbol Device:C
- added D510, D511, D512, D513: BAT46WJ, Diode_SMD:D_SOD-323F, symbol Diode:BAT46
- added R526, R532, R543, R544, R545, R546: 100k, Resistor_SMD:R_0603_1608Metric, symbol Device:R
- added R530: 220k, Resistor_SMD:R_0603_1608Metric, symbol Device:R
- added R531: 1M, Resistor_SMD:R_0603_1608Metric, symbol Device:R
- added R534: 5.76k, Resistor_SMD:R_0603_1608Metric, symbol Device:R
- added R535, R537, R539, R541: 10k, Resistor_SMD:R_0603_1608Metric, symbol Device:R
- added R536: 274k, Resistor_SMD:R_0603_1608Metric, symbol Device:R
- added R538: 1.37k, Resistor_SMD:R_0603_1608Metric, symbol Device:R
- added R540: 80.6k, Resistor_SMD:R_0603_1608Metric, symbol Device:R
- added R542: 182k, Resistor_SMD:R_0603_1608Metric, symbol Device:R
- added U507, U508: LM2901B-Q1, Package_SO:SOIC-14_3.9x8.7mm_P1.27mm, symbol Comparator:LM2901
- R501: value 6.8k -> 2.2k; MPN ERJ-3EKF6801V -> ERJ-3EKF2201V
- R504: value 180k -> 174k; MPN TNPW0603180KBEEA -> TNPW0603174KBEEA
- R514: value 10k -> 100k; MPN ERJ-3EKF1002V -> ERJ-3EKF1003V
- R518: value 2.2k -> 4.7k; MPN ERJ-3EKF2201V -> ERJ-3EKF4701V
Connections:
- net +3V3: now also D512.2 (A), R543.1; no longer R514.1, U503.8 (VCC)
- net AUX12: now also C515.1, C517.1, R544.1, R545.1, R546.1, U507.3 (V+), U508.3 (V+)
- net GND: now also C514.2, C515.2, C516.2, C517.2, C518.2, C519.2, C521.2, C522.2, C523.2, R530.2, R535.2, R537.2, R539.2, R541.2, U507.12 (V-), U508.10 (-), U508.12 (V-); no longer U506.10 (-), U506.8 (-)
- net K_IN: now also D510.2 (A), D511.2 (A)
- net LATCH_Q: now also R532.1
- net LATCH_QN: now also D510.1 (K)
- net NTC_P1: now also U508.4 (-)
- net NTC_P2: now also U508.8 (-)
- net OVP_TRIP_N: now also U506.13, U506.14, U507.1
- net PERMIT: now also U508.14, U508.2
- net RESET_N: no longer U503.6 (~{CLR})
- net VREF2V5: now also R526.1, R534.1, R536.1, R538.1
- net VTH2V0: now also R526.2, U507.11 (+), U507.9 (+), U508.6 (-)
- net VTH_OC: no longer U506.11 (+), U506.9 (+)
- new net AUX_IN: R540.1
- new net AUX_PG: D511.1 (K), R542.1, R543.2, U508.1
- new net AUX_PGS: C519.1, R540.2, R541.1, R542.2, U508.7 (+)
- new net BURST_N: R544.2, U507.2
- new net CLR_N: C523.1, D513.2 (A), R531.2, U503.6 (~{CLR})
- new net DCX_CS: U507.6 (-)
- new net LATCH_SNS: R532.2
- new net LATCH_VCC: C521.1, C522.1, D512.1 (K), D513.1 (K), R514.1, R530.1, R531.1, U503.8 (VCC)
- new net LIM: U507.4 (-)
- new net ONT_H: U506.8 (-)
- new net ONT_L: U506.10 (-)
- new net PVA_OVS: U507.8 (-)
- new net PVA_OV_N: R545.2, U507.14
- new net PVB_OVS: U507.10 (-)
- new net PVB_OV_N: R546.2, U507.13
- new net VTH_BURST: U507.5 (+)
- new net VTH_DOC: C516.1, R536.2, R537.1, U507.7 (+)
- new net VTH_ONT: C514.1, R534.2, R535.1, U506.11 (+), U506.9 (+)
- new net VTH_OPEN: C518.1, R538.2, R539.1, U508.11 (+), U508.5 (+), U508.9 (+)
- no-connect marks 6 -> 5
Other:
- moved on the sheet: C502, C503, C504, C505, C506, C508, C509, C510, C511, C512, C513, D501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
